File: src/kicad/board/power2.kicad_sch (KiCad schematic)
At the start: 12 parts, among them Q1 DMG2301L, SW6 Enable BAT, U3 BQ25172

Commit message: update wip
Parts:
- removed D2: D_Schottky, symbol Device:D_Schottky
- added C8: 10uF, Capacitor_SMD:C_0805_2012Metric, symbol Device:C
- D1: footprint (none) -> LED_SMD:LED_0805_2012Metric
- U3: footprint (none) -> Library:BQ25172
Connections:
- net GND: now also C8.2
- net OUT: no longer BT1.1 (+), Q1.3 (D), U3.8 (OUT)
- new net: BT1.1 (+), C8.1, Q1.3 (D), U3.8 (OUT)
Other:
- moved on the sheet: BT1, Q1, SW6

Commit message: update
Parts:
- removed SW6: Enable BAT, Button_Switch_SMD:SW_DIP_SPSTx01_Slide_9.78x4.72mm_W8.61mm_P2.54mm, symbol Switch:SW_SPST
- added J4, J5: Conn_01x02_Male, Connector_PinHeader_2.54mm:PinHeader_1x02_P2.54mm_Vertical, symbol Connector:Conn_01x02_Male
- C7, C8: Vendor (none) -> C15850
- D1: Vendor (none) -> C84256
- Q1: value DMG2301L -> DMG2305UX; Vendor (none) -> C2940629
- R10: value 10K -> 1K; Vendor (none) -> C17513
- R11: value 8.2K -> 20K; Vendor (none) -> C17544
- R12: value 36K -> 20K; Vendor (none) -> C17544
- R8: Vendor (none) -> C17513
- R9: Vendor (none) -> C17414
- U3: footprint Library:BQ25172 -> Package_SON:WSON-8-1EP_2x2mm_P0.5mm_EP0.9x1.6mm; Vendor (none) -> C5189434
Connections:
- net OUT: now also J5.1 (Pin_1)
- net USB_VBUS: now also J4.2 (Pin_2); no longer C7.1, Q1.1 (G), R10.1, U3.1 (IN)
- net at Q1.2 (S): now also J5.2 (Pin_2)
- new net: C7.1, J4.1 (Pin_1), Q1.1 (G), R10.1, U3.1 (IN)
Changed lines of the file:
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@@
+    (stroke (width 0) (type default) (color 0 0 0 0))
+  )
+  (wire (pts (xy 201.93 109.22) (xy 213.36 109.22))
     (stroke (width 0) (type default) (color 0 0 0 0))
   )
@@
     (stroke (width 0) (type default) (color 0 0 0 0))
   )
-  (wire (pts (xy 207.01 109.22) (xy 214.63 109.22))
-    (stroke (width 0) (type default) (color 0 0 0 0))
-  )
   (wire (pts (xy 190.5 93.98) (xy 190.5 95.25))
     (stroke (width 0) (type default) (color 0 0 0 0))
@@
     (stroke (width 0) (type default) (color 0 0 0 0))
   )
-  (wire (pts (xy 190.5 109.22) (xy 196.85 109.22))
+  (wire (pts (xy 190.5 109.22) (xy 199.39 109.22))
     (stroke (width 0) (type default) (color 0 0 0 0))
   )
@@
     (stroke (width 0) (type default) (color 0 0 0 0))
   )
+  (wire (pts (xy 93.98 82.55) (xy 105.41 82.55))
+    (stroke (width 0) (type default) (color 0 0 0 0))
+  )
   (wire (pts (xy 110.49 110.49) (xy 116.84 110.49))
     (stroke (width 0) (type default) (color 0 0 0 0))
@@
     (stroke (width 0) (type default) (color 0 0 0 0))
   )
-  (wire (pts (xy 102.87 82.55) (xy 105.41 82.55))
+  (wire (pts (xy 87.63 82.55) (xy 91.44 82.55))
     (stroke (width 0) (type default) (color 0 0 0 0))
   )
@@
     (stroke (width 0) (type default) (color 0 0 0 0))
   )
-  (hierarchical_label "OUT" (shape input) (at 214.63 109.22 0)
+  (hierarchical_label "OUT" (shape input) (at 213.36 109.22 0)
     (effects (font (size 1.27 1.27)) (justify left))
   )
-  (hierarchical_label "USB_VBUS" (shape input) (at 102.87 82.55 180)
+  (hierarchical_label "USB_VBUS" (shape input) (at 87.63 82.55 180)
     (effects (font (size 1.27 1.27)) (justify right))
   )
@@
       (effects (font (size 1.27 1.27)) (justify left))
     )
-    (property "Value" "DMG2301L" (id 1) (at 190.5 95.25 0)
+    (property "Value" "DMG2305UX" (id 1) (at 190.5 95.25 0)
       (effects (font (size 1.27 1.27)) (justify left))
     )
@@
       (effects (font (size 1.27 1.27) italic) (justify left) hide)
     )
-    (property "Datasheet" "https://www.diodes.com/assets/Datasheets/DMG2301L.pdf" (id 3) (at 187.96 100.33 0)
+    (property "Datasheet" "https://www.diodes.com/assets/Datasheets/DMG2305UX.pdf" (id 3) (at 187.96 100.33 0)
       (effects (font (size 1.27 1.27)) (justify left) hide)
     )
+    (property "Vendor" "C2940629" (id 4) (at 187.96 100.33 0)
+      (effects (font (size 1.27 1.27)) hide)
+    )
     (pin "1")
     (pin "2")
@@
       (effects (font (size 1.27 1.27)) (justify left))
     )
-    (property "Value" "36K" (id 1) (at 158.75 105.41 90)
+    (property "Value" "20K" (id 1) (at 158.75 105.41 90)
       (effects (font (size 1.27 1.27)) (justify left))
     )
@@
     )
     (property "Datasheet" "~" (id 3) (at 158.75 102.87 0)
+      (effects (font (size 1.27 1.27)) hide)
+    )
+    (property "Vendor" "C17544" (id 4) (at 158.75 102.87 0)
       (effects (font (size 1.27 1.27)) hide)
     )
@@
       (effects (font (size 1.27 1.27)) hide)
     )
+    (property "Vendor" "C84256" (id 4) (at 139.7 82.55 0)
+      (effects (font (size 1.27 1.27)) hide)
+    )
+    (pin "1")
+    (pin "2")
+  )
+  (symbol (lib_id "Connector:Conn_01x02_Male") (at 93.98 77.47 270) (unit 1)
+    (in_bom yes) (on_board yes) (fields_autoplaced)
+    (property "Reference" "J4" (id 0) (at 95.25 76.8349 90)
+      (effects (font (size 1.27 1.27)) (justify left))
+    )
+    (property "Value" "Conn_01x02_Male" (id 1) (at 95.25 79.3749 90)
+      (effects (font (size 1.27 1.27)) (justify left))
+    )
+    (property "Footprint" "Connector_PinHeader_2.54mm:PinHeader_1x02_P2.54mm_Vertical" (id 2) (at 93.98 77.47 0)
+      (effects (font (size 1.27 1.27)) hide)
+    )
+    (property "Datasheet" "~" (id 3) (at 93.98 77.47 0)
+      (effects (font (size 1.27 1.27)) hide)
+    )
     (pin "1")
     (pin "2")
@@
     (in_bom yes) (on_board yes)
     (property "Reference" "R10" (id 0) (at 129.54 80.01 90))
-    (property "Value" "10K" (id 1) (at 129.54 82.55 90))
+    (property "Value" "1K" (id 1) (at 129.54 82.55 90))
     (property "Footprint" "Resistor_SMD:R_0805_2012Metric" (id 2) (at 129.54 84.328 90)
       (effects (font (size 1.27 1.27)) hide)
@@
       (effects (font (size 1.27 1.27)) hide)
     )
+    (property "Vendor" "C17513" (id 4) (at 129.54 82.55 0)
+      (effects (font (size 1.27 1.27)) hide)
+    )
     (pin "1")
     (pin "2")
@@
     )
     (property "Datasheet" "~" (id 3) (at 166.37 102.87 0)
+      (effects (font (size 1.27 1.27)) hide)
+    )
+    (property "Vendor" "C15850" (id 4) (at 166.37 102.87 0)
       (effects (font (size 1.27 1.27)) hide)
     )
@@
       (effects (font (size 1.27 1.27)) hide)
     )
-    (pin "1")
-    (pin "2")
-  )
-  (symbol (lib_id "Switch:SW_SPST") (at 201.93 109.22 0) (unit 1)
-    (in_bom yes) (on_board yes) (fields_autoplaced)
-    (property "Reference" "SW6" (id 0) (at 201.93 102.87 0))
-    (property "Value" "Enable BAT" (id 1) (at 201.93 105.41 0))
-    (property "Footprint" "Button_Switch_SMD:SW_DIP_SPSTx01_Slide_9.78x4.72mm_W8.61mm_P2.54mm" (id 2) (at 201.93 109.22 0)
-      (effects (font (size 1.27 1.27)) hide)
-    )
-    (property "Datasheet" "~" (id 3) (at 201.93 109.22 0)
+    (property "Vendor" "C17414" (id 4) (at 116.84 102.87 0)
       (effects (font (size 1.27 1.27)) hide)
     )
@@
       (effects (font (size 1.27 1.27)) (justify left))
     )
-    (property "Value" "8.2K" (id 1) (at 152.4 105.41 90)
+    (property "Value" "20K" (id 1) (at 152.4 105.41 90)
       (effects (font (size 1.27 1.27)) (justify left))
     )
@@
     )
     (property "Datasheet" "~" (id 3) (at 152.4 102.87 0)
+      (effects (font (size 1.27 1.27)) hide)
+    )
+    (property "Vendor" "C17544" (id 4) (at 152.4 102.87 0)
       (effects (font (size 1.27 1.27)) hide)
     )
@@
       (effects (font (size 1.27 1.27)) hide)
     )
+    (property "Vendor" "C17513" (id 4) (at 110.49 102.87 0)
+      (effects (font (size 1.27 1.27)) hide)
+    )
+    (pin "1")
+    (pin "2")
+  )
+  (symbol (lib_id "Connector:Conn_01x02_Male") (at 201.93 104.14 270) (unit 1)
+    (in_bom yes) (on_board yes) (fields_autoplaced)
+    (property "Reference" "J5" (id 0) (at 203.2 103.5049 90)
+      (effects (font (size 1.27 1.27)) (justify left))
+    )
+    (property "Value" "Conn_01x02_Male" (id 1) (at 203.2 106.0449 90)
+      (effects (font (size 1.27 1.27)) (justify left))
+    )
+    (property "Footprint" "Connector_PinHeader_2.54mm:PinHeader_1x02_P2.54mm_Vertical" (id 2) (at 201.93 104.14 0)
+      (effects (font (size 1.27 1.27)) hide)
+    )
+    (property "Datasheet" "~" (id 3) (at 201.93 104.14 0)
+      (effects (font (size 1.27 1.27)) hide)
+    )
     (pin "1")
     (pin "2")
@@
     )
     (property "Datasheet" "~" (id 3) (at 105.41 99.06 0)
+      (effects (font (size 1.27 1.27)) hide)
+    )
+    (property "Vendor" "C15850" (id 4) (at 105.41 99.06 0)
       (effects (font (size 1.27 1.27)) hide)
     )
@@
     (property "Reference" "U3" (id 0) (at 134.62 87.63 0))
     (property "Value" "BQ25172" (id 1) (at 134.62 90.17 0))
-    (property "Footprint" "Library:BQ25172" (id 2) (at 132.08 96.52 0)
+    (property "Footprint" "Package_SON:WSON-8-1EP_2x2mm_P0.5mm_EP0.9x1.6mm" (id 2) (at 132.08 96.52 0)
       (effects (font (size 1.27 1.27)) hide)
     )
@@
       (effects (font (size 1.27 1.27)) hide)
     )
+    (property "Vendor" "C5189434" (id 4) (at 134.62 99.06 0)
+      (effects (font (size 1.27 1.27)) hide)
+    )

Commit message: update
Parts:
- BT1: footprint Battery:BatteryHolder_Keystone_2479_3xAAA -> Battery:BatteryHolder_Keystone_2462_2xAA
- renumbered C7 to C5, C8 to C6, J4 to J5, J5 to J6, R8 to R17, R9 to R18, R10 to R19, R11 to R20, R12 to R21, U3 to U4
Other:
- note added: "https://datasheets.raspberrypi.com/pico/pico-datasheet.pdf#powerchain-section"
Changed lines of the file:
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@@
   (junction (at 158.75 110.49) (diameter 0) (color 0 0 0 0)
   )
+  (junction (at 105.41 93.98) (diameter 0) (color 0 0 0 0)
+  )
   (junction (at 166.37 93.98) (diameter 0) (color 0 0 0 0)
   )
@@
     (stroke (width 0) (type default) (color 0 0 0 0))
   )
-  (wire (pts (xy 105.41 82.55) (xy 105.41 95.25))
+  (wire (pts (xy 105.41 82.55) (xy 105.41 93.98))
     (stroke (width 0) (type default) (color 0 0 0 0))
   )
@@
     (stroke (width 0) (type default) (color 0 0 0 0))
   )
-  (wire (pts (xy 113.03 93.98) (xy 125.73 93.98))
-    (stroke (width 0) (type default) (color 0 0 0 0))
-  )
   (wire (pts (xy 147.32 101.6) (xy 147.32 82.55))
     (stroke (width 0) (type default) (color 0 0 0 0))
   )
+  (wire (pts (xy 105.41 93.98) (xy 125.73 93.98))
+    (stroke (width 0) (type default) (color 0 0 0 0))
+  )
   (wire (pts (xy 190.5 93.98) (xy 190.5 95.25))
     (stroke (width 0) (type default) (color 0 0 0 0))
@@
     (stroke (width 0) (type default) (color 0 0 0 0))
   )
-  (wire (pts (xy 113.03 82.55) (xy 113.03 93.98))
-    (stroke (width 0) (type default) (color 0 0 0 0))
-  )
   (wire (pts (xy 190.5 109.22) (xy 199.39 109.22))
     (stroke (width 0) (type default) (color 0 0 0 0))
@@
     (stroke (width 0) (type default) (color 0 0 0 0))
   )
+  (wire (pts (xy 105.41 93.98) (xy 105.41 95.25))
+    (stroke (width 0) (type default) (color 0 0 0 0))
+  )
   (wire (pts (xy 166.37 93.98) (xy 166.37 99.06))
     (stroke (width 0) (type default) (color 0 0 0 0))
@@
   (wire (pts (xy 133.35 82.55) (xy 135.89 82.55))
     (stroke (width 0) (type default) (color 0 0 0 0))
+  )
+  (text "https://datasheets.raspberrypi.com/pico/pico-datasheet.pdf#powerchain-section"
+    (at 85.09 68.58 0)
+    (effects (font (size 1.27 1.27) italic) (justify left bottom))
   )
   (hierarchical_label "OUT" (shape input) (at 213.36 109.22 0)
@@
   (symbol (lib_id "Device:R") (at 158.75 102.87 0) (unit 1)
     (in_bom yes) (on_board yes)
-    (property "Reference" "R12" (id 0) (at 156.21 106.68 0)
+    (property "Reference" "R21" (id 0) (at 156.21 106.68 0)
       (effects (font (size 1.27 1.27)) (justify left))
     )
@@
   (symbol (lib_id "power:GND") (at 134.62 113.03 0) (unit 1)
     (in_bom yes) (on_board yes) (fields_autoplaced)
-    (property "Reference" "#PWR0109" (id 0) (at 134.62 119.38 0)
+    (property "Reference" "#PWR029" (id 0) (at 134.62 119.38 0)
       (effects (font (size 1.27 1.27)) hide)
     )
@@
   (symbol (lib_id "Connector:Conn_01x02_Male") (at 93.98 77.47 270) (unit 1)
     (in_bom yes) (on_board yes) (fields_autoplaced)
-    (property "Reference" "J4" (id 0) (at 95.25 76.8349 90)
+    (property "Reference" "J5" (id 0) (at 95.25 76.8349 90)
       (effects (font (size 1.27 1.27)) (justify left))
     )
@@
   (symbol (lib_id "Device:R") (at 129.54 82.55 90) (unit 1)
     (in_bom yes) (on_board yes)
-    (property "Reference" "R10" (id 0) (at 129.54 80.01 90))
+    (property "Reference" "R19" (id 0) (at 129.54 80.01 90))
     (property "Value" "1K" (id 1) (at 129.54 82.55 90))
     (property "Footprint" "Resistor_SMD:R_0805_2012Metric" (id 2) (at 129.54 84.328 90)
@@
   (symbol (lib_id "Device:C") (at 166.37 102.87 0) (unit 1)
     (in_bom yes) (on_board yes)
-    (property "Reference" "C8" (id 0) (at 162.56 100.33 0)
+    (property "Reference" "C6" (id 0) (at 162.56 100.33 0)
       (effects (font (size 1.27 1.27)) (justify left))
     )
@@
   (symbol (lib_id "Device:R") (at 116.84 102.87 180) (unit 1)
     (in_bom yes) (on_board yes)
-    (property "Reference" "R9" (id 0) (at 119.38 101.6 0))
+    (property "Reference" "R18" (id 0) (at 119.38 101.6 0))
     (property "Value" "10K" (id 1) (at 116.84 102.87 90))
     (property "Footprint" "Resistor_SMD:R_0805_2012Metric" (id 2) (at 118.618 102.87 90)
@@
       (effects (font (size 1.27 1.27)) (justify left))
     )
-    (property "Footprint" "Battery:BatteryHolder_Keystone_2479_3xAAA" (id 2) (at 173.99 100.076 90)
+    (property "Footprint" "Battery:BatteryHolder_Keystone_2462_2xAA" (id 2) (at 173.99 100.076 90)
       (effects (font (size 1.27 1.27)) hide)
     )
@@
   (symbol (lib_id "Device:R") (at 152.4 102.87 0) (unit 1)
     (in_bom yes) (on_board yes)
-    (property "Reference" "R11" (id 0) (at 151.13 106.68 0)
+    (property "Reference" "R20" (id 0) (at 151.13 106.68 0)
       (effects (font (size 1.27 1.27)) (justify left))
     )
@@
   (symbol (lib_id "Device:R") (at 110.49 102.87 180) (unit 1)
     (in_bom yes) (on_board yes)
-    (property "Reference" "R8" (id 0) (at 113.03 101.6 0))
+    (property "Reference" "R17" (id 0) (at 113.03 101.6 0))
     (property "Value" "1K" (id 1) (at 110.49 102.87 90))
     (property "Footprint" "Resistor_SMD:R_0805_2012Metric" (id 2) (at 112.268 102.87 90)
@@
   (symbol (lib_id "Connector:Conn_01x02_Male") (at 201.93 104.14 270) (unit 1)
     (in_bom yes) (on_board yes) (fields_autoplaced)
-    (property "Reference" "J5" (id 0) (at 203.2 103.5049 90)
+    (property "Reference" "J6" (id 0) (at 203.2 103.5049 90)
       (effects (font (size 1.27 1.27)) (justify left))
     )
@@
   (symbol (lib_id "Device:C") (at 105.41 99.06 0) (unit 1)
     (in_bom yes) (on_board yes)
-    (property "Reference" "C7" (id 0) (at 101.6 96.52 0)
+    (property "Reference" "C5" (id 0) (at 101.6 96.52 0)
       (effects (font (size 1.27 1.27)) (justify left))
     )
@@
   (symbol (lib_id "project_library:BQ25172") (at 134.62 99.06 0) (unit 1)
     (in_bom yes) (on_board yes)
-    (property "Reference" "U3" (id 0) (at 134.62 87.63 0))
+    (property "Reference" "U4" (id 0) (at 134.62 87.63 0))
     (property "Value" "BQ25172" (id 1) (at 134.62 90.17 0))
     (property "Footprint" "Package_SON:WSON-8-1EP_2x2mm_P0.5mm_EP0.9x1.6mm" (id 2) (at 132.08 96.52 0)

Commit message: update
Parts:
- R20, R21: Vendor C17544 -> C4328
Changed lines of the file:
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@@
       (effects (font (size 1.27 1.27)) hide)
     )
-    (property "Vendor" "C17544" (id 4) (at 158.75 102.87 0)
+    (property "Vendor" "C4328" (id 4) (at 158.75 102.87 0)
       (effects (font (size 1.27 1.27)) hide)
     )
@@
       (effects (font (size 1.27 1.27)) hide)
     )
-    (property "Vendor" "C17544" (id 4) (at 152.4 102.87 0)
+    (property "Vendor" "C4328" (id 4) (at 152.4 102.87 0)
       (effects (font (size 1.27 1.27)) hide)
     )
