File: src/kicad/board/power2.kicad_sch (KiCad schematic)
At the start: 21 parts, among them Q1 DMG2305UX, U4 BQ25172, U5 TLV61070A, U6 XC6206P332MR

Commit message: update
Parts:
- added D?: B5819W SL, Diode_SMD:D_SOD-123, symbol Diode:1N5819
- U6: Vendor (none) -> C5446
Connections:
- net USB_VBUS: now also D?.2 (A); no longer C5.1, Q1.1 (G), R23.1, U4.1 (IN)
- new net: C5.1, D?.1 (K), Q1.1 (G), R23.1, U4.1 (IN)
Changed lines of the file:
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@@
     (stroke (width 0) (type default) (color 0 0 0 0))
   )
-  (wire (pts (xy 100.33 45.72) (xy 107.95 45.72))
+  (wire (pts (xy 101.6 45.72) (xy 107.95 45.72))
+    (stroke (width 0) (type default) (color 0 0 0 0))
+  )
+  (wire (pts (xy 88.9 45.72) (xy 93.98 45.72))
     (stroke (width 0) (type default) (color 0 0 0 0))
   )
@@
     (effects (font (size 1.27 1.27)) (justify left))
   )
-  (hierarchical_label "USB_VBUS" (shape input) (at 100.33 45.72 180)
+  (hierarchical_label "USB_VBUS" (shape input) (at 88.9 45.72 180)
     (effects (font (size 1.27 1.27)) (justify right))
   )
@@
       (effects (font (size 1.27 1.27)) hide)
     )
+    (property "Vendor" "C5446" (id 4) (at 185.42 132.08 0)
+      (effects (font (size 1.27 1.27)) hide)
+    )
     (pin "1")
     (pin "2")
@@
       (effects (font (size 1.27 1.27)) hide)
     )
+    (pin "1")
+    (pin "2")
+  )
+  (symbol (lib_id "Diode:1N5819") (at 97.79 45.72 180) (unit 1)
+    (in_bom yes) (on_board yes) (fields_autoplaced)
+    (property "Reference" "D?" (id 0) (at 98.1075 39.37 0))
+    (property "Value" "B5819W SL" (id 1) (at 98.1075 41.91 0))
+    (property "Footprint" "Diode_SMD:D_SOD-123" (id 2) (at 97.79 41.275 0)
+      (effects (font (size 1.27 1.27)) hide)
+    )
+    (property "Datasheet" "" (id 3) (at 97.79 45.72 0)
+      (effects (font (size 1.27 1.27)) hide)
+    )
+    (property "Vendor" "C8598" (id 4) (at 97.79 45.72 0)
+      (effects (font (size 1.27 1.27)) hide)
+    )

Commit message: update, schematic should be done
Parts:
- R11: renamed from R21; footprint Resistor_SMD:R_0805_2012Metric -> Resistor_SMD:R_0603_1608Metric; Vendor C17513 -> C21190
- R12: renamed from R22; footprint Resistor_SMD:R_0805_2012Metric -> Resistor_SMD:R_0603_1608Metric; Vendor C17414 -> C25804
- gave numbers to parts that had none: 2
- renumbered C5 to C4, C6 to C5, C7 to C6, C8 to C7, C9 to C8, C10 to C9, D2 to D5, R23 to R13, R24 to R14, R25 to R15, R26 to R16, R27 to R17, U4 to U2, U5 to U3, U6 to U4
Changed lines of the file:
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@@
   (symbol (lib_id "Device:C") (at 198.12 137.16 0) (unit 1)
     (in_bom yes) (on_board yes)
-    (property "Reference" "C10" (id 0) (at 194.31 134.62 0)
+    (property "Reference" "C9" (id 0) (at 194.31 134.62 0)
       (effects (font (size 1.27 1.27)) (justify left))
     )
@@
   (symbol (lib_id "Device:C") (at 120.65 105.41 0) (unit 1)
     (in_bom yes) (on_board yes) (fields_autoplaced)
-    (property "Reference" "C6" (id 0) (at 123.825 104.1399 0)
+    (property "Reference" "C5" (id 0) (at 123.825 104.1399 0)
       (effects (font (size 1.27 1.27)) (justify left))
     )
@@
   (symbol (lib_id "Regulator_Linear:XC6206PxxxMR") (at 185.42 132.08 0) (unit 1)
     (in_bom yes) (on_board yes) (fields_autoplaced)
-    (property "Reference" "U6" (id 0) (at 185.42 124.46 0))
+    (property "Reference" "U4" (id 0) (at 185.42 124.46 0))
     (property "Value" "XC6206P332MR" (id 1) (at 185.42 127 0))
     (property "Footprint" "Package_TO_SOT_SMD:SOT-23-3" (id 2) (at 185.42 126.365 0)
@@
   (symbol (lib_id "Device:R") (at 161.29 66.04 0) (unit 1)
     (in_bom yes) (on_board yes)
-    (property "Reference" "R27" (id 0) (at 158.75 69.85 0)
+    (property "Reference" "R17" (id 0) (at 158.75 69.85 0)
       (effects (font (size 1.27 1.27)) (justify left))
     )
@@
   (symbol (lib_id "Device:R") (at 153.035 133.35 0) (unit 1)
     (in_bom yes) (on_board yes) (fields_autoplaced)
-    (property "Reference" "R25" (id 0) (at 154.94 132.0799 0)
+    (property "Reference" "R15" (id 0) (at 154.94 132.0799 0)
       (effects (font (size 1.27 1.27)) (justify left))
     )
@@
   (symbol (lib_id "power:GND") (at 137.16 76.2 0) (unit 1)
     (in_bom yes) (on_board yes) (fields_autoplaced)
-    (property "Reference" "#PWR011" (id 0) (at 137.16 82.55 0)
+    (property "Reference" "#PWR012" (id 0) (at 137.16 82.55 0)
       (effects (font (size 1.27 1.27)) hide)
     )
@@
   (symbol (lib_id "Device:LED") (at 142.24 45.72 180) (unit 1)
     (in_bom yes) (on_board yes)
-    (property "Reference" "D2" (id 0) (at 140.97 43.18 0))
+    (property "Reference" "D5" (id 0) (at 140.97 43.18 0))
     (property "Value" "CHARGE_LED" (id 1) (at 142.24 48.26 0))
     (property "Footprint" "LED_SMD:LED_0805_2012Metric" (id 2) (at 142.24 45.72 0)
@@
   (symbol (lib_id "Device:R") (at 132.08 45.72 90) (unit 1)
     (in_bom yes) (on_board yes)
-    (property "Reference" "R23" (id 0) (at 132.08 43.18 90))
+    (property "Reference" "R13" (id 0) (at 132.08 43.18 90))
     (property "Value" "2K7" (id 1) (at 132.08 45.72 90))
     (property "Footprint" "Resistor_SMD:R_0805_2012Metric" (id 2) (at 132.08 47.498 90)
@@
   (symbol (lib_id "Connector_Generic:Conn_01x02") (at 201.93 77.47 270) (unit 1)
     (in_bom yes) (on_board yes) (fields_autoplaced)
-    (property "Reference" "J?" (id 0) (at 204.47 76.1999 90)
+    (property "Reference" "J6" (id 0) (at 204.47 76.1999 90)
       (effects (font (size 1.27 1.27)) (justify left))
     )
@@
   (symbol (lib_id "power:GND") (at 163.195 140.335 0) (unit 1)
     (in_bom yes) (on_board yes) (fields_autoplaced)
-    (property "Reference" "#PWR012" (id 0) (at 163.195 146.685 0)
+    (property "Reference" "#PWR013" (id 0) (at 163.195 146.685 0)
       (effects (font (size 1.27 1.27)) hide)
     )
@@
   (symbol (lib_id "Device:C") (at 168.91 66.04 0) (unit 1)
     (in_bom yes) (on_board yes)
-    (property "Reference" "C8" (id 0) (at 165.1 63.5 0)
+    (property "Reference" "C7" (id 0) (at 165.1 63.5 0)
       (effects (font (size 1.27 1.27)) (justify left))
     )
@@
   (symbol (lib_id "Device:R") (at 119.38 66.04 180) (unit 1)
     (in_bom yes) (on_board yes)
-    (property "Reference" "R22" (id 0) (at 121.92 64.77 0))
+    (property "Reference" "R12" (id 0) (at 121.92 64.77 0))
     (property "Value" "10K" (id 1) (at 119.38 66.04 90))
-    (property "Footprint" "Resistor_SMD:R_0805_2012Metric" (id 2) (at 121.158 66.04 90)
+    (property "Footprint" "Resistor_SMD:R_0603_1608Metric" (id 2) (at 121.158 66.04 90)
       (effects (font (size 1.27 1.27)) hide)
     )
@@
       (effects (font (size 1.27 1.27)) hide)
     )
-    (property "Vendor" "C17414" (id 4) (at 119.38 66.04 0)
+    (property "Vendor" "C25804" (id 4) (at 119.38 66.04 0)
       (effects (font (size 1.27 1.27)) hide)
     )
@@
   (symbol (lib_id "power:GND") (at 120.65 120.65 0) (unit 1)
     (in_bom yes) (on_board yes)
-    (property "Reference" "#PWR010" (id 0) (at 120.65 127 0)
+    (property "Reference" "#PWR011" (id 0) (at 120.65 127 0)
       (effects (font (size 1.27 1.27)) hide)
     )
@@
   (symbol (lib_id "project_library:TLV61070A") (at 139.7 118.11 0) (unit 1)
     (in_bom yes) (on_board yes) (fields_autoplaced)
-    (property "Reference" "U5" (id 0) (at 139.7 106.68 0))
+    (property "Reference" "U3" (id 0) (at 139.7 106.68 0))
     (property "Value" "TLV61070A" (id 1) (at 139.7 109.22 0))
     (property "Footprint" "Package_SO:TSOP-6_1.65x3.05mm_P0.95mm" (id 2) (at 138.684 117.856 0)
@@
   (symbol (lib_id "power:GND") (at 185.42 144.78 0) (unit 1)
     (in_bom yes) (on_board yes)
-    (property "Reference" "#PWR013" (id 0) (at 185.42 151.13 0)
+    (property "Reference" "#PWR014" (id 0) (at 185.42 151.13 0)
       (effects (font (size 1.27 1.27)) hide)
     )
@@
   (symbol (lib_id "Device:C") (at 175.26 137.16 0) (unit 1)
     (in_bom yes) (on_board yes)
-    (property "Reference" "C9" (id 0) (at 171.45 134.62 0)
+    (property "Reference" "C8" (id 0) (at 171.45 134.62 0)
       (effects (font (size 1.27 1.27)) (justify left))
     )
@@
   (symbol (lib_id "Diode:1N5819") (at 97.79 45.72 180) (unit 1)
     (in_bom yes) (on_board yes) (fields_autoplaced)
-    (property "Reference" "D?" (id 0) (at 98.1075 39.37 0))
+    (property "Reference" "D4" (id 0) (at 98.1075 39.37 0))
     (property "Value" "B5819W SL" (id 1) (at 98.1075 41.91 0))
     (property "Footprint" "Diode_SMD:D_SOD-123" (id 2) (at 97.79 41.275 0)
@@
   (symbol (lib_id "Device:R") (at 154.94 66.04 0) (unit 1)
     (in_bom yes) (on_board yes)
-    (property "Reference" "R26" (id 0) (at 153.67 69.85 0)
+    (property "Reference" "R16" (id 0) (at 153.67 69.85 0)
       (effects (font (size 1.27 1.27)) (justify left))
     )
@@
   (symbol (lib_id "Device:R") (at 153.035 123.19 0) (unit 1)
     (in_bom yes) (on_board yes)
-    (property "Reference" "R24" (id 0) (at 154.94 121.92 0)
+    (property "Reference" "R14" (id 0) (at 154.94 121.92 0)
       (effects (font (size 1.27 1.27)) (justify left))
     )
@@
   (symbol (lib_id "Device:R") (at 113.03 66.04 180) (unit 1)
     (in_bom yes) (on_board yes)
-    (property "Reference" "R21" (id 0) (at 115.57 64.77 0))
+    (property "Reference" "R11" (id 0) (at 115.57 64.77 0))
     (property "Value" "1K" (id 1) (at 113.03 66.04 90))
-    (property "Footprint" "Resistor_SMD:R_0805_2012Metric" (id 2) (at 114.808 66.04 90)
+    (property "Footprint" "Resistor_SMD:R_0603_1608Metric" (id 2) (at 114.808 66.04 90)
       (effects (font (size 1.27 1.27)) hide)
     )
@@
       (effects (font (size 1.27 1.27)) hide)
     )
-    (property "Vendor" "C17513" (id 4) (at 113.03 66.04 0)
+    (property "Vendor" "C21190" (id 4) (at 113.03 66.04 0)
       (effects (font (size 1.27 1.27)) hide)
     )
@@
   (symbol (lib_id "Device:C") (at 107.95 62.23 0) (unit 1)
     (in_bom yes) (on_board yes)
-    (property "Reference" "C5" (id 0) (at 104.14 59.69 0)
+    (property "Reference" "C4" (id 0) (at 104.14 59.69 0)
       (effects (font (size 1.27 1.27)) (justify left))
     )
@@
   (symbol (lib_id "Device:C") (at 163.195 124.46 0) (unit 1)
     (in_bom yes) (on_board yes) (fields_autoplaced)
-    (property "Reference" "C7" (id 0) (at 167.005 123.1899 0)
+    (property "Reference" "C6" (id 0) (at 167.005 123.1899 0)
       (effects (font (size 1.27 1.27)) (justify left))
     )
@@
   (symbol (lib_id "project_library:BQ25172") (at 137.16 62.23 0) (unit 1)
     (in_bom yes) (on_board yes)
-    (property "Reference" "U4" (id 0) (at 137.16 50.8 0))
+    (property "Reference" "U2" (id 0) (at 137.16 50.8 0))
     (property "Value" "BQ25172" (id 1) (at 137.16 53.34 0))
     (property "Footprint" "Package_SON:WSON-8-1EP_2x2mm_P0.5mm_EP0.9x1.6mm" (id 2) (at 134.62 59.69 0)

Commit message: wip
Parts:
- C4, C5, C7, C8, C9: footprint Capacitor_SMD:C_0805_2012Metric -> Capacitor_SMD:C_0603_1608Metric; Vendor C15850 -> C19702
- C6: footprint Capacitor_SMD:C_0805_2012Metric -> Capacitor_SMD:C_0603_1608Metric; Vendor C45783 -> C59461
- R13, R15: footprint Resistor_SMD:R_0805_2012Metric -> Resistor_SMD:R_0603_1608Metric; Vendor C17530 -> C13167
- R16: footprint Resistor_SMD:R_0805_2012Metric -> Resistor_SMD:R_0603_1608Metric; Vendor C17593 -> C22967
- R17: footprint Resistor_SMD:R_0805_2012Metric -> Resistor_SMD:R_0603_1608Metric; Vendor C4328 -> C4184
Changed lines of the file:
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@@
       (effects (font (size 1.27 1.27)) (justify left))
     )
-    (property "Footprint" "Capacitor_SMD:C_0805_2012Metric" (id 2) (at 199.0852 140.97 0)
+    (property "Footprint" "Capacitor_SMD:C_0603_1608Metric" (id 2) (at 199.0852 140.97 0)
       (effects (font (size 1.27 1.27)) hide)
     )
@@
       (effects (font (size 1.27 1.27)) hide)
     )
-    (property "Vendor" "C15850" (id 4) (at 198.12 137.16 0)
+    (property "Vendor" "C19702" (id 4) (at 198.12 137.16 0)
       (effects (font (size 1.27 1.27)) hide)
     )
@@
       (effects (font (size 1.27 1.27)) (justify left))
     )
-    (property "Footprint" "Capacitor_SMD:C_0805_2012Metric" (id 2) (at 121.6152 109.22 0)
+    (property "Footprint" "Capacitor_SMD:C_0603_1608Metric" (id 2) (at 121.6152 109.22 0)
       (effects (font (size 1.27 1.27)) hide)
     )
@@
       (effects (font (size 1.27 1.27)) hide)
     )
-    (property "Vendor" "C15850" (id 4) (at 120.65 105.41 0)
+    (property "Vendor" "C19702" (id 4) (at 120.65 105.41 0)
       (effects (font (size 1.27 1.27)) hide)
     )
@@
       (effects (font (size 1.27 1.27)) (justify left))
     )
-    (property "Footprint" "Resistor_SMD:R_0805_2012Metric" (id 2) (at 159.512 66.04 90)
+    (property "Footprint" "Resistor_SMD:R_0603_1608Metric" (id 2) (at 159.512 66.04 90)
       (effects (font (size 1.27 1.27)) hide)
     )
@@
       (effects (font (size 1.27 1.27)) hide)
     )
-    (property "Vendor" "C4328" (id 4) (at 161.29 66.04 0)
+    (property "Vendor" "C4184" (id 4) (at 161.29 66.04 0)
       (effects (font (size 1.27 1.27)) hide)
     )
@@
       (effects (font (size 1.27 1.27)) (justify left))
     )
-    (property "Footprint" "Resistor_SMD:R_0805_2012Metric" (id 2) (at 151.257 133.35 90)
+    (property "Footprint" "Resistor_SMD:R_0603_1608Metric" (id 2) (at 151.257 133.35 90)
       (effects (font (size 1.27 1.27)) hide)
     )
@@
       (effects (font (size 1.27 1.27)) hide)
     )
-    (property "Vendor" "C17530" (id 4) (at 153.035 133.35 0)
+    (property "Vendor" "C13167" (id 4) (at 153.035 133.35 0)
       (effects (font (size 1.27 1.27)) hide)
     )
@@
     (property "Reference" "R13" (id 0) (at 132.08 43.18 90))
     (property "Value" "2K7" (id 1) (at 132.08 45.72 90))
-    (property "Footprint" "Resistor_SMD:R_0805_2012Metric" (id 2) (at 132.08 47.498 90)
+    (property "Footprint" "Resistor_SMD:R_0603_1608Metric" (id 2) (at 132.08 47.498 90)
       (effects (font (size 1.27 1.27)) hide)
     )
@@
       (effects (font (size 1.27 1.27)) hide)
     )
-    (property "Vendor" "C17530" (id 4) (at 132.08 45.72 0)
+    (property "Vendor" "C13167" (id 4) (at 132.08 45.72 0)
       (effects (font (size 1.27 1.27)) hide)
     )
@@
       (effects (font (size 1.27 1.27)) (justify left))
     )
-    (property "Footprint" "Capacitor_SMD:C_0805_2012Metric" (id 2) (at 169.8752 69.85 0)
+    (property "Footprint" "Capacitor_SMD:C_0603_1608Metric" (id 2) (at 169.8752 69.85 0)
       (effects (font (size 1.27 1.27)) hide)
     )
@@
       (effects (font (size 1.27 1.27)) hide)
     )
-    (property "Vendor" "C15850" (id 4) (at 168.91 66.04 0)
+    (property "Vendor" "C19702" (id 4) (at 168.91 66.04 0)
       (effects (font (size 1.27 1.27)) hide)
     )
@@
       (effects (font (size 1.27 1.27)) (justify left))
     )
-    (property "Footprint" "Capacitor_SMD:C_0805_2012Metric" (id 2) (at 176.2252 140.97 0)
+    (property "Footprint" "Capacitor_SMD:C_0603_1608Metric" (id 2) (at 176.2252 140.97 0)
       (effects (font (size 1.27 1.27)) hide)
     )
@@
       (effects (font (size 1.27 1.27)) hide)
     )
-    (property "Vendor" "C15850" (id 4) (at 175.26 137.16 0)
+    (property "Vendor" "C19702" (id 4) (at 175.26 137.16 0)
       (effects (font (size 1.27 1.27)) hide)
     )
@@
       (effects (font (size 1.27 1.27)) (justify left))
     )
-    (property "Footprint" "Resistor_SMD:R_0805_2012Metric" (id 2) (at 153.162 66.04 90)
+    (property "Footprint" "Resistor_SMD:R_0603_1608Metric" (id 2) (at 153.162 66.04 90)
       (effects (font (size 1.27 1.27)) hide)
     )
@@
       (effects (font (size 1.27 1.27)) hide)
     )
-    (property "Vendor" "C17593" (id 4) (at 154.94 66.04 0)
+    (property "Vendor" "C22967" (id 4) (at 154.94 66.04 0)
       (effects (font (size 1.27 1.27)) hide)
     )
@@
       (effects (font (size 1.27 1.27)) (justify left))
     )
-    (property "Footprint" "Capacitor_SMD:C_0805_2012Metric" (id 2) (at 108.9152 66.04 0)
+    (property "Footprint" "Capacitor_SMD:C_0603_1608Metric" (id 2) (at 108.9152 66.04 0)
       (effects (font (size 1.27 1.27)) hide)
     )
@@
       (effects (font (size 1.27 1.27)) hide)
     )
-    (property "Vendor" "C15850" (id 4) (at 107.95 62.23 0)
+    (property "Vendor" "C19702" (id 4) (at 107.95 62.23 0)
       (effects (font (size 1.27 1.27)) hide)
     )
@@
       (effects (font (size 1.27 1.27)) (justify left))
     )
-    (property "Footprint" "Capacitor_SMD:C_0805_2012Metric" (id 2) (at 164.1602 128.27 0)
+    (property "Footprint" "Capacitor_SMD:C_0603_1608Metric" (id 2) (at 164.1602 128.27 0)
       (effects (font (size 1.27 1.27)) hide)
     )
@@
       (effects (font (size 1.27 1.27)) hide)
     )
-    (property "Vendor" "C45783" (id 4) (at 163.195 124.46 0)
-      (effects (font (size 1.27 1.27)) hide)
-    )
+    (property "Vendor" "C59461" (id 4) (at 163.195 124.46 0)
+      (effects (font (size 1.27 1.27)) hide)
+    )

Commit message: update
Parts:
- R17: value 20K -> 27K; Vendor C4184 -> C22967
Other:
- note added: "27K -> 2-cell + intermittent charge"
Changed lines of the file:
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@@
+    (effects (font (size 1.27 1.27)) (justify left bottom))
+  )
+  (text "27K -> 2-cell + intermittent charge\n" (at 158.75 73.66 90)
     (effects (font (size 1.27 1.27)) (justify left bottom))
   )
@@
       (effects (font (size 1.27 1.27)) (justify left))
     )
-    (property "Value" "20K" (id 1) (at 161.29 68.58 90)
+    (property "Value" "27K" (id 1) (at 161.29 68.58 90)
       (effects (font (size 1.27 1.27)) (justify left))
     )
@@
       (effects (font (size 1.27 1.27)) hide)
     )
-    (property "Vendor" "C4184" (id 4) (at 161.29 66.04 0)
+    (property "Vendor" "C22967" (id 4) (at 161.29 66.04 0)
       (effects (font (size 1.27 1.27)) hide)
     )
