File: src/kicad/board/input.kicad_sch (KiCad schematic)
At the start: 7 parts, among them SW1 SW_Keyboard, SW2 SW_Keyboard, SW3 RotEncoder_S, SW4 SW_Keyboard, SW5 SW_Keyboard

Commit message: update, schematic should be done
Parts:
- SW1, SW2, SW4, SW5: footprint Button_Switch_Keyboard:SW_Cherry_MX_1.00u_PCB -> Library:Kailh_socket_MX
- gave numbers to parts that had none: 2
Changed lines of the file:
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@@
   (symbol (lib_id "Device:C") (at 99.06 62.23 0) (unit 1)
     (in_bom yes) (on_board yes) (fields_autoplaced)
-    (property "Reference" "C?" (id 0) (at 102.87 60.9599 0)
+    (property "Reference" "C3" (id 0) (at 102.87 60.9599 0)
       (effects (font (size 1.27 1.27)) (justify left))
     )
@@
     (property "Reference" "SW5" (id 0) (at 207.01 83.82 0))
     (property "Value" "SW_Keyboard" (id 1) (at 207.01 86.36 0))
-    (property "Footprint" "Button_Switch_Keyboard:SW_Cherry_MX_1.00u_PCB" (id 2) (at 210.82 86.36 0)
+    (property "Footprint" "Library:Kailh_socket_MX" (id 2) (at 210.82 86.36 0)
       (effects (font (size 1.27 1.27)) hide)
     )
@@
     (property "Reference" "SW2" (id 0) (at 182.88 83.82 0))
     (property "Value" "SW_Keyboard" (id 1) (at 182.88 86.36 0))
-    (property "Footprint" "Button_Switch_Keyboard:SW_Cherry_MX_1.00u_PCB" (id 2) (at 184.15 86.36 0)
+    (property "Footprint" "Library:Kailh_socket_MX" (id 2) (at 184.15 86.36 0)
       (effects (font (size 1.27 1.27)) hide)
     )
@@
     (property "Reference" "SW4" (id 0) (at 207.01 68.58 0))
     (property "Value" "SW_Keyboard" (id 1) (at 207.01 71.12 0))
-    (property "Footprint" "Button_Switch_Keyboard:SW_Cherry_MX_1.00u_PCB" (id 2) (at 210.82 71.12 0)
+    (property "Footprint" "Library:Kailh_socket_MX" (id 2) (at 210.82 71.12 0)
       (effects (font (size 1.27 1.27)) hide)
     )
@@
   (symbol (lib_id "Interface_Expansion:MCP23017_ML") (at 118.11 96.52 0) (unit 1)
     (in_bom yes) (on_board yes) (fields_autoplaced)
-    (property "Reference" "U?" (id 0) (at 120.1294 68.58 0)
+    (property "Reference" "U1" (id 0) (at 120.1294 68.58 0)
       (effects (font (size 1.27 1.27)) (justify left))
     )
@@
     (property "Reference" "SW1" (id 0) (at 181.61 68.58 0))
     (property "Value" "SW_Keyboard" (id 1) (at 181.61 71.12 0))
-    (property "Footprint" "Button_Switch_Keyboard:SW_Cherry_MX_1.00u_PCB" (id 2) (at 184.15 71.12 0)
+    (property "Footprint" "Library:Kailh_socket_MX" (id 2) (at 184.15 71.12 0)
       (effects (font (size 1.27 1.27)) hide)
     )

Commit message: wip
Parts:
- C3: value 0.1uF -> 100nF; footprint Capacitor_SMD:C_0805_2012Metric -> Capacitor_SMD:C_0603_1608Metric; Vendor C28233 -> C14663
Changed lines of the file:
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@@
       (effects (font (size 1.27 1.27)) (justify left))
     )
-    (property "Value" "0.1uF" (id 1) (at 102.87 63.4999 0)
+    (property "Value" "100nF" (id 1) (at 102.87 63.4999 0)
       (effects (font (size 1.27 1.27)) (justify left))
     )
-    (property "Footprint" "Capacitor_SMD:C_0805_2012Metric" (id 2) (at 100.0252 66.04 0)
+    (property "Footprint" "Capacitor_SMD:C_0603_1608Metric" (id 2) (at 100.0252 66.04 0)
       (effects (font (size 1.27 1.27)) hide)
     )
@@
       (effects (font (size 1.27 1.27)) hide)
     )
-    (property "Vendor" "C28233" (id 4) (at 99.06 62.23 0)
+    (property "Vendor" "C14663" (id 4) (at 99.06 62.23 0)
       (effects (font (size 1.27 1.27)) hide)
     )

Commit message: update
Parts:
- C3: footprint Capacitor_SMD:C_0603_1608Metric -> Capacitor_SMD:C_0402_1005Metric; Vendor C14663 -> C307331
Changed lines of the file:
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@@
       (effects (font (size 1.27 1.27)) (justify left))
     )
-    (property "Footprint" "Capacitor_SMD:C_0603_1608Metric" (id 2) (at 100.0252 66.04 0)
+    (property "Footprint" "Capacitor_SMD:C_0402_1005Metric" (id 2) (at 100.0252 66.04 0)
       (effects (font (size 1.27 1.27)) hide)
     )
@@
       (effects (font (size 1.27 1.27)) hide)
     )
-    (property "Vendor" "C14663" (id 4) (at 99.06 62.23 0)
+    (property "Vendor" "C307331" (id 4) (at 99.06 62.23 0)
       (effects (font (size 1.27 1.27)) hide)
     )
