File: src/kicad/board/rp2040.kicad_sch (KiCad schematic)
At the start: 21 parts

Commit message: update
Parts:
- C15, C16, C17, C18, C19, C20, C21, C22, C23, C24, C25, C26, C27, C28: renamed from C?; footprint (none) -> Capacitor_SMD:C_0805_2012Metric
- R28, R29: renamed from R?; footprint (none) -> Resistor_SMD:R_0805_2012Metric; Vendor (none) -> C17513
- R30: renamed from R?; footprint (none) -> Resistor_SMD:R_0805_2012Metric; Vendor (none) -> C17414
- SW7: renamed from SW?; Vendor (none) -> C318884
- gave numbers to parts that had none: 3

Commit message: update
Parts:
- C15, C16: footprint Capacitor_SMD:C_0805_2012Metric -> Capacitor_SMD:C_0603_1608Metric; Vendor (none) -> C107045
- C17, C18, C20, C22, C23, C24, C25, C26, C27, C28: footprint Capacitor_SMD:C_0805_2012Metric -> Capacitor_SMD:C_0603_1608Metric; Vendor (none) -> C14663
- C19, C21: footprint Capacitor_SMD:C_0805_2012Metric -> Capacitor_SMD:C_0603_1608Metric; Vendor (none) -> C15849
- SW7: footprint (none) -> Button_Switch_SMD:SW_SPST_SKQG_WithoutStem
- U8: Vendor (none) -> C2040
Connections:
- net RUN: no longer names the net of U8.26 (RUN)
- no-connect marks 0 -> 1
Other:
- note added: "Default: Internal pullup to enable"
Changed lines of the file:
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@@
   (junction (at 87.63 40.64) (diameter 0) (color 0 0 0 0)
   )
+  (no_connect (at 67.31 74.93))
   (wire (pts (xy 64.77 82.55) (xy 67.31 82.55))
     (stroke (width 0) (type default) (color 0 0 0 0))
@@
   )
   (wire (pts (xy 73.66 50.8) (xy 73.66 52.07))
-    (stroke (width 0) (type default) (color 0 0 0 0))
-  )
-  (wire (pts (xy 63.5 74.93) (xy 67.31 74.93))
     (stroke (width 0) (type default) (color 0 0 0 0))
   )
@@
     (effects (font (size 1.27 1.27)) (justify left bottom))
   )
+  (text "Default: Internal pullup to enable" (at 33.02 76.2 0)
+    (effects (font (size 1.27 1.27)) (justify left bottom))
+  )
   (label "QSPI_SD0" (at 66.04 97.79 180)
     (effects (font (size 1.27 1.27)) (justify right bottom))
@@
   (hierarchical_label "GPIO24" (shape bidirectional) (at 119.38 135.89 0)
     (effects (font (size 1.27 1.27)) (justify left))
-  )
-  (hierarchical_label "RUN" (shape input) (at 63.5 74.93 180)
-    (effects (font (size 1.27 1.27)) (justify right))
   )
   (hierarchical_label "GPIO17" (shape bidirectional) (at 119.38 118.11 0)
@@
       (effects (font (size 1.27 1.27)) (justify left))
     )
-    (property "Footprint" "Capacitor_SMD:C_0805_2012Metric" (id 2) (at 256.2352 104.14 0)
+    (property "Footprint" "Capacitor_SMD:C_0603_1608Metric" (id 2) (at 256.2352 104.14 0)
       (effects (font (size 1.27 1.27)) hide)
     )
@@
       (effects (font (size 1.27 1.27)) hide)
     )
+    (property "Vendor" "C14663" (id 4) (at 255.27 100.33 0)
+      (effects (font (size 1.27 1.27)) hide)
+    )
     (pin "1")
     (pin "2")
@@
       (effects (font (size 1.27 1.27)) (justify left))
     )
-    (property "Footprint" "Capacitor_SMD:C_0805_2012Metric" (id 2) (at 64.4652 50.8 0)
+    (property "Footprint" "Capacitor_SMD:C_0603_1608Metric" (id 2) (at 64.4652 50.8 0)
       (effects (font (size 1.27 1.27)) hide)
     )
@@
       (effects (font (size 1.27 1.27)) hide)
     )
+    (property "Vendor" "C14663" (id 4) (at 63.5 46.99 0)
+      (effects (font (size 1.27 1.27)) hide)
+    )
     (pin "1")
     (pin "2")
@@
       (effects (font (size 1.27 1.27)) (justify left))
     )
-    (property "Footprint" "Capacitor_SMD:C_0805_2012Metric" (id 2) (at 74.6252 50.8 0)
+    (property "Footprint" "Capacitor_SMD:C_0603_1608Metric" (id 2) (at 74.6252 50.8 0)
       (effects (font (size 1.27 1.27)) hide)
     )
@@
       (effects (font (size 1.27 1.27)) hide)
     )
+    (property "Vendor" "C14663" (id 4) (at 73.66 46.99 0)
+      (effects (font (size 1.27 1.27)) hide)
+    )
     (pin "1")
     (pin "2")
@@
       (effects (font (size 1.27 1.27)) (justify left))
     )
-    (property "Footprint" "Capacitor_SMD:C_0805_2012Metric" (id 2) (at 79.7052 63.5 0)
+    (property "Footprint" "Capacitor_SMD:C_0603_1608Metric" (id 2) (at 79.7052 63.5 0)
       (effects (font (size 1.27 1.27)) hide)
     )
@@
       (effects (font (size 1.27 1.27)) hide)
     )
+    (property "Vendor" "C15849" (id 4) (at 78.74 59.69 0)
+      (effects (font (size 1.27 1.27)) hide)
+    )
     (pin "1")
     (pin "2")
@@
       (effects (font (size 1.27 1.27)) (justify left))
     )
-    (property "Footprint" "Capacitor_SMD:C_0805_2012Metric" (id 2) (at 140.6652 49.53 0)
+    (property "Footprint" "Capacitor_SMD:C_0603_1608Metric" (id 2) (at 140.6652 49.53 0)
       (effects (font (size 1.27 1.27)) hide)
     )
     (property "Datasheet" "~" (id 3) (at 139.7 45.72 0)
+      (effects (font (size 1.27 1.27)) hide)
+    )
+    (property "Vendor" "C14663" (id 4) (at 139.7 45.72 0)
       (effects (font (size 1.27 1.27)) hide)
     )
@@
     (property "Reference" "C15" (id 0) (at 39.37 116.84 90))
     (property "Value" "27pF" (id 1) (at 39.37 124.46 90))
-    (property "Footprint" "Capacitor_SMD:C_0805_2012Metric" (id 2) (at 43.18 119.6848 0)
+    (property "Footprint" "Capacitor_SMD:C_0603_1608Metric" (id 2) (at 43.18 119.6848 0)
       (effects (font (size 1.27 1.27)) hide)
     )
     (property "Datasheet" "~" (id 3) (at 39.37 120.65 0)
+      (effects (font (size 1.27 1.27)) hide)
+    )
+    (property "Vendor" "C107045" (id 4) (at 39.37 120.65 0)
       (effects (font (size 1.27 1.27)) hide)
     )
@@
       (effects (font (size 1.27 1.27)) (justify left))
     )
-    (property "Footprint" "Capacitor_SMD:C_0805_2012Metric" (id 2) (at 113.9952 49.53 0)
+    (property "Footprint" "Capacitor_SMD:C_0603_1608Metric" (id 2) (at 113.9952 49.53 0)
       (effects (font (size 1.27 1.27)) hide)
     )
     (property "Datasheet" "~" (id 3) (at 113.03 45.72 0)
+      (effects (font (size 1.27 1.27)) hide)
+    )
+    (property "Vendor" "C14663" (id 4) (at 113.03 45.72 0)
       (effects (font (size 1.27 1.27)) hide)
     )
@@
     (property "Reference" "C16" (id 0) (at 39.37 127 90))
     (property "Value" "27pF" (id 1) (at 39.37 134.62 90))
-    (property "Footprint" "Capacitor_SMD:C_0805_2012Metric" (id 2) (at 35.56 131.7752 0)
+    (property "Footprint" "Capacitor_SMD:C_0603_1608Metric" (id 2) (at 35.56 131.7752 0)
       (effects (font (size 1.27 1.27)) hide)
     )
     (property "Datasheet" "~" (id 3) (at 39.37 130.81 0)
+      (effects (font (size 1.27 1.27)) hide)
+    )
+    (property "Vendor" "C107045" (id 4) (at 39.37 130.81 0)
       (effects (font (size 1.27 1.27)) hide)
     )
@@
   )
   (symbol (lib_id "Switch:SW_Push") (at 168.91 106.68 0) (unit 1)
-    (in_bom yes) (on_board yes)
+    (in_bom yes) (on_board yes) (fields_autoplaced)
     (property "Reference" "SW7" (id 0) (at 168.91 99.06 0))
     (property "Value" "BOOTSEL" (id 1) (at 168.91 101.6 0))
-    (property "Footprint" "" (id 2) (at 168.91 101.6 0)
+    (property "Footprint" "Button_Switch_SMD:SW_SPST_SKQG_WithoutStem" (id 2) (at 168.91 101.6 0)
       (effects (font (size 1.27 1.27)) hide)
     )
@@
       (effects (font (size 1.27 1.27)) (justify left))
     )
-    (property "Footprint" "Capacitor_SMD:C_0805_2012Metric" (id 2) (at 115.2652 63.5 0)
+    (property "Footprint" "Capacitor_SMD:C_0603_1608Metric" (id 2) (at 115.2652 63.5 0)
       (effects (font (size 1.27 1.27)) hide)
     )
@@
       (effects (font (size 1.27 1.27)) hide)
     )
+    (property "Vendor" "C15849" (id 4) (at 114.3 59.69 0)
+      (effects (font (size 1.27 1.27)) hide)
+    )
     (pin "1")
     (pin "2")
@@
     )
     (property "Datasheet" "https://datasheets.raspberrypi.com/rp2040/rp2040-datasheet.pdf" (id 3) (at 92.71 113.03 0)
+      (effects (font (size 1.27 1.27)) hide)
+    )
+    (property "Vendor" "C2040" (id 4) (at 92.71 113.03 0)
       (effects (font (size 1.27 1.27)) hide)
     )
@@
       (effects (font (size 1.27 1.27)) (justify left))
     )
-    (property "Footprint" "Capacitor_SMD:C_0805_2012Metric" (id 2) (at 158.4452 49.53 0)
+    (property "Footprint" "Capacitor_SMD:C_0603_1608Metric" (id 2) (at 158.4452 49.53 0)
       (effects (font (size 1.27 1.27)) hide)
     )
     (property "Datasheet" "~" (id 3) (at 157.48 45.72 0)
+      (effects (font (size 1.27 1.27)) hide)
+    )
+    (property "Vendor" "C14663" (id 4) (at 157.48 45.72 0)
       (effects (font (size 1.27 1.27)) hide)
     )
@@
       (effects (font (size 1.27 1.27)) (justify left))
     )
-    (property "Footprint" "Capacitor_SMD:C_0805_2012Metric" (id 2) (at 167.3352 49.53 0)
+    (property "Footprint" "Capacitor_SMD:C_0603_1608Metric" (id 2) (at 167.3352 49.53 0)
       (effects (font (size 1.27 1.27)) hide)
     )
@@
       (effects (font (size 1.27 1.27)) hide)
     )
+    (property "Vendor" "C14663" (id 4) (at 166.37 45.72 0)
+      (effects (font (size 1.27 1.27)) hide)
+    )
     (pin "1")
     (pin "2")
@@
       (effects (font (size 1.27 1.27)) (justify left))
     )
-    (property "Footprint" "Capacitor_SMD:C_0805_2012Metric" (id 2) (at 122.8852 49.53 0)
+    (property "Footprint" "Capacitor_SMD:C_0603_1608Metric" (id 2) (at 122.8852 49.53 0)
       (effects (font (size 1.27 1.27)) hide)
     )
@@
       (effects (font (size 1.27 1.27)) hide)
     )
+    (property "Vendor" "C14663" (id 4) (at 121.92 45.72 0)
+      (effects (font (size 1.27 1.27)) hide)
+    )
     (pin "1")
     (pin "2")
@@
       (effects (font (size 1.27 1.27)) (justify left))
     )
-    (property "Footprint" "Capacitor_SMD:C_0805_2012Metric" (id 2) (at 149.5552 49.53 0)
+    (property "Footprint" "Capacitor_SMD:C_0603_1608Metric" (id 2) (at 149.5552 49.53 0)
       (effects (font (size 1.27 1.27)) hide)
     )
@@
       (effects (font (size 1.27 1.27)) hide)
     )
+    (property "Vendor" "C14663" (id 4) (at 148.59 45.72 0)
+      (effects (font (size 1.27 1.27)) hide)
+    )
     (pin "1")
     (pin "2")
@@
       (effects (font (size 1.27 1.27)) (justify left))
     )
-    (property "Footprint" "Capacitor_SMD:C_0805_2012Metric" (id 2) (at 131.7752 49.53 0)
+    (property "Footprint" "Capacitor_SMD:C_0603_1608Metric" (id 2) (at 131.7752 49.53 0)
       (effects (font (size 1.27 1.27)) hide)
     )
@@
       (effects (font (size 1.27 1.27)) hide)
     )
+    (property "Vendor" "C14663" (id 4) (at 130.81 45.72 0)
+      (effects (font (size 1.27 1.27)) hide)
+    )

Commit message: update, schematic should be done
Parts:
- R18: renamed from R28; footprint Resistor_SMD:R_0805_2012Metric -> Resistor_SMD:R_0603_1608Metric; Vendor C17513 -> C21190
- R19: renamed from R29; footprint Resistor_SMD:R_0805_2012Metric -> Resistor_SMD:R_0603_1608Metric; Vendor C17513 -> C21190
- R20: renamed from R30; footprint Resistor_SMD:R_0805_2012Metric -> Resistor_SMD:R_0603_1608Metric; Vendor C17414 -> C25804
- renumbered C15 to C14, C16 to C15, C17 to C16, C18 to C17, C19 to C18, C20 to C19, C21 to C20, C22 to C21, C23 to C22, C24 to C23, C25 to C24, C26 to C25, C27 to C26, C28 to C27, SW7 to SW6, U8 to U6, U9 to U7
Connections:
- net +3.3V: no longer C14.1, C15.2, C16.2, C17.2, C18.2, C19.2, C20.2, C21.2, C22.2, C23.2, C24.2, C25.2, C26.2, C27.2, SW6.1, U6.19 (TESTEN), U6.57 (GND), U7.4 (GND), Y1.2, Y1.4
- new net GND: C14.1, C15.2, C16.2, C17.2, C18.2, C19.2, C20.2, C21.2, C22.2, C23.2, C24.2, C25.2, C26.2, C27.2, SW6.1, U6.19 (TESTEN), U6.57 (GND), U7.4 (GND), Y1.2, Y1.4

Commit message: update
Parts:
- C16, C17, C19, C21, C22, C23, C24, C25, C26, C27: footprint Capacitor_SMD:C_0603_1608Metric -> Capacitor_SMD:C_0402_1005Metric; Vendor C14663 -> C307331
- C18, C20: footprint Capacitor_SMD:C_0603_1608Metric -> Capacitor_SMD:C_0402_1005Metric; Vendor C15849 -> C52923
Changed lines of the file:
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@@
       (effects (font (size 1.27 1.27)) (justify left))
     )
-    (property "Footprint" "Capacitor_SMD:C_0603_1608Metric" (id 2) (at 256.2352 104.14 0)
+    (property "Footprint" "Capacitor_SMD:C_0402_1005Metric" (id 2) (at 256.2352 104.14 0)
       (effects (font (size 1.27 1.27)) hide)
     )
@@
       (effects (font (size 1.27 1.27)) hide)
     )
-    (property "Vendor" "C14663" (id 4) (at 255.27 100.33 0)
+    (property "Vendor" "C307331" (id 4) (at 255.27 100.33 0)
       (effects (font (size 1.27 1.27)) hide)
     )
@@
       (effects (font (size 1.27 1.27)) (justify left))
     )
-    (property "Footprint" "Capacitor_SMD:C_0603_1608Metric" (id 2) (at 64.4652 50.8 0)
+    (property "Footprint" "Capacitor_SMD:C_0402_1005Metric" (id 2) (at 64.4652 50.8 0)
       (effects (font (size 1.27 1.27)) hide)
     )
@@
       (effects (font (size 1.27 1.27)) hide)
     )
-    (property "Vendor" "C14663" (id 4) (at 63.5 46.99 0)
+    (property "Vendor" "C307331" (id 4) (at 63.5 46.99 0)
       (effects (font (size 1.27 1.27)) hide)
     )
@@
       (effects (font (size 1.27 1.27)) (justify left))
     )
-    (property "Footprint" "Capacitor_SMD:C_0603_1608Metric" (id 2) (at 74.6252 50.8 0)
+    (property "Footprint" "Capacitor_SMD:C_0402_1005Metric" (id 2) (at 74.6252 50.8 0)
       (effects (font (size 1.27 1.27)) hide)
     )
@@
       (effects (font (size 1.27 1.27)) hide)
     )
-    (property "Vendor" "C14663" (id 4) (at 73.66 46.99 0)
+    (property "Vendor" "C307331" (id 4) (at 73.66 46.99 0)
       (effects (font (size 1.27 1.27)) hide)
     )
@@
       (effects (font (size 1.27 1.27)) (justify left))
     )
-    (property "Footprint" "Capacitor_SMD:C_0603_1608Metric" (id 2) (at 79.7052 63.5 0)
+    (property "Footprint" "Capacitor_SMD:C_0402_1005Metric" (id 2) (at 79.7052 63.5 0)
       (effects (font (size 1.27 1.27)) hide)
     )
@@
       (effects (font (size 1.27 1.27)) hide)
     )
-    (property "Vendor" "C15849" (id 4) (at 78.74 59.69 0)
+    (property "Vendor" "C52923" (id 4) (at 78.74 59.69 0)
       (effects (font (size 1.27 1.27)) hide)
     )
@@
       (effects (font (size 1.27 1.27)) (justify left))
     )
-    (property "Footprint" "Capacitor_SMD:C_0603_1608Metric" (id 2) (at 140.6652 49.53 0)
+    (property "Footprint" "Capacitor_SMD:C_0402_1005Metric" (id 2) (at 140.6652 49.53 0)
       (effects (font (size 1.27 1.27)) hide)
     )
@@
       (effects (font (size 1.27 1.27)) hide)
     )
-    (property "Vendor" "C14663" (id 4) (at 139.7 45.72 0)
+    (property "Vendor" "C307331" (id 4) (at 139.7 45.72 0)
       (effects (font (size 1.27 1.27)) hide)
     )
@@
       (effects (font (size 1.27 1.27)) (justify left))
     )
-    (property "Footprint" "Capacitor_SMD:C_0603_1608Metric" (id 2) (at 113.9952 49.53 0)
+    (property "Footprint" "Capacitor_SMD:C_0402_1005Metric" (id 2) (at 113.9952 49.53 0)
       (effects (font (size 1.27 1.27)) hide)
     )
@@
       (effects (font (size 1.27 1.27)) hide)
     )
-    (property "Vendor" "C14663" (id 4) (at 113.03 45.72 0)
+    (property "Vendor" "C307331" (id 4) (at 113.03 45.72 0)
       (effects (font (size 1.27 1.27)) hide)
     )
@@
       (effects (font (size 1.27 1.27)) (justify left))
     )
-    (property "Footprint" "Capacitor_SMD:C_0603_1608Metric" (id 2) (at 115.2652 63.5 0)
+    (property "Footprint" "Capacitor_SMD:C_0402_1005Metric" (id 2) (at 115.2652 63.5 0)
       (effects (font (size 1.27 1.27)) hide)
     )
@@
       (effects (font (size 1.27 1.27)) hide)
     )
-    (property "Vendor" "C15849" (id 4) (at 114.3 59.69 0)
+    (property "Vendor" "C52923" (id 4) (at 114.3 59.69 0)
       (effects (font (size 1.27 1.27)) hide)
     )
@@
       (effects (font (size 1.27 1.27)) (justify left))
     )
-    (property "Footprint" "Capacitor_SMD:C_0603_1608Metric" (id 2) (at 158.4452 49.53 0)
+    (property "Footprint" "Capacitor_SMD:C_0402_1005Metric" (id 2) (at 158.4452 49.53 0)
       (effects (font (size 1.27 1.27)) hide)
     )
@@
       (effects (font (size 1.27 1.27)) hide)
     )
-    (property "Vendor" "C14663" (id 4) (at 157.48 45.72 0)
+    (property "Vendor" "C307331" (id 4) (at 157.48 45.72 0)
       (effects (font (size 1.27 1.27)) hide)
     )
@@
       (effects (font (size 1.27 1.27)) (justify left))
     )
-    (property "Footprint" "Capacitor_SMD:C_0603_1608Metric" (id 2) (at 167.3352 49.53 0)
+    (property "Footprint" "Capacitor_SMD:C_0402_1005Metric" (id 2) (at 167.3352 49.53 0)
       (effects (font (size 1.27 1.27)) hide)
     )
@@
       (effects (font (size 1.27 1.27)) hide)
     )
-    (property "Vendor" "C14663" (id 4) (at 166.37 45.72 0)
+    (property "Vendor" "C307331" (id 4) (at 166.37 45.72 0)
       (effects (font (size 1.27 1.27)) hide)
     )
@@
       (effects (font (size 1.27 1.27)) (justify left))
     )
-    (property "Footprint" "Capacitor_SMD:C_0603_1608Metric" (id 2) (at 122.8852 49.53 0)
+    (property "Footprint" "Capacitor_SMD:C_0402_1005Metric" (id 2) (at 122.8852 49.53 0)
       (effects (font (size 1.27 1.27)) hide)
     )
@@
       (effects (font (size 1.27 1.27)) hide)
     )
-    (property "Vendor" "C14663" (id 4) (at 121.92 45.72 0)
+    (property "Vendor" "C307331" (id 4) (at 121.92 45.72 0)
       (effects (font (size 1.27 1.27)) hide)
     )
@@
       (effects (font (size 1.27 1.27)) (justify left))
     )
-    (property "Footprint" "Capacitor_SMD:C_0603_1608Metric" (id 2) (at 149.5552 49.53 0)
+    (property "Footprint" "Capacitor_SMD:C_0402_1005Metric" (id 2) (at 149.5552 49.53 0)
       (effects (font (size 1.27 1.27)) hide)
     )
@@
       (effects (font (size 1.27 1.27)) hide)
     )
-    (property "Vendor" "C14663" (id 4) (at 148.59 45.72 0)
+    (property "Vendor" "C307331" (id 4) (at 148.59 45.72 0)
       (effects (font (size 1.27 1.27)) hide)
     )
@@
       (effects (font (size 1.27 1.27)) (justify left))
     )
-    (property "Footprint" "Capacitor_SMD:C_0603_1608Metric" (id 2) (at 131.7752 49.53 0)
+    (property "Footprint" "Capacitor_SMD:C_0402_1005Metric" (id 2) (at 131.7752 49.53 0)
       (effects (font (size 1.27 1.27)) hide)
     )
@@
       (effects (font (size 1.27 1.27)) hide)
     )
-    (property "Vendor" "C14663" (id 4) (at 130.81 45.72 0)
-      (effects (font (size 1.27 1.27)) hide)
-    )
+    (property "Vendor" "C307331" (id 4) (at 130.81 45.72 0)
+      (effects (font (size 1.27 1.27)) hide)
+    )
