File: src/kicad/board/board.kicad_pcb (KiCad board)
At the start: 2 copper layers, 109.4 x 83.4 mm, 50 parts, among them J1 Screw_Terminal_Speaker, J2 Micro_SD_Card_Det, Q1 DMG2301L, SW1 SW_Keyboard, SW2 SW_Keyboard, SW3 RotEncoder_S, SW4 SW_Keyboard, SW5 SW_Keyboard, SW6 Enable BAT, U1 Pico, U2 MAX98357, U3 BQ25172, U5 74HC4051, U6 4072

Commit message: update wip
Parts:
- moved SW5 8.71 mm to (193.4, 97.8)
- moved SW4 8.63 mm to (173.9, 97.8)
- moved SW1 8.62 mm to (135.2, 97.8)
- moved SW2 8.52 mm to (154.7, 97.9)
- moved R19 5.32 mm to (109.8, 94.5)
- moved R20 5.32 mm to (105.1, 94.5)
- moved R21 5.25 mm to (107.5, 94.7)
- moved SW6 5.21 mm to (159.4, 79.2)
- moved SW3 4.96 mm to (105.8, 103.1)
- moved D1 3.71 mm to (163.4, 69.8)
- moved BT1 1.52 mm to (199.6, 42.9)
- moved R9 0.32 mm to (156.6, 66.4)
- moved R8 0.29 mm to (154.6, 66.4)
- turned R10 to -90 degrees
Routing:
- net +3.3V: track 19.0 -> 135.6 mm, vias 0 -> 20
- net B3: track 41.9 -> 118.7 mm, vias 2 -> 3
- net /Power2/USB_VBUS: track 0.00 -> 64.4 mm, vias 0 -> 2
- net B1: track 40.4 -> 99.7 mm, vias 3 -> 4
- net Net-(BT1-Pad1): track 0.00 -> 55.9 mm
- net B2: track 35.9 -> 81.5 mm, vias 2 -> 3
- net Net-(Q1-Pad2): track 0.00 -> 27.4 mm
- net GP26: track 0.00 -> 25.1 mm
- net GP27: track 0.00 -> 24.5 mm
- net B0: track 40.7 -> 63.4 mm, vias 2 -> 3
- net GP28: track 0.00 -> 16.8 mm, vias 0 -> 2
- net Net-(FB2-Pad1): track 0.00 -> 12.4 mm
- net Net-(C3-Pad1): track 0.00 -> 11.2 mm
- net GND: track 21.7 -> 32.3 mm, vias 4 -> 36
- net VDD: track 0.00 -> 10.3 mm
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- added copper zone on F.Cu, net +3.3V
- added copper zone on B.Cu, net GND
- added copper zone on F.Cu, net VDD
Other:
- board size 109.4 x 83.4 mm -> 108.2 x 77.1 mm

Commit message: update
Parts:
- removed R1: 1M, Resistor_SMD:R_0805_2012Metric
- removed SW6: Enable BAT, Button_Switch_SMD:SW_DIP_SPSTx01_Slide_9.78x4.72mm_W8.61mm_P2.54mm
- added J3: Conn_01x06, Connector_PinHeader_2.54mm:PinHeader_1x06_P2.54mm_Vertical, F.Cu at (163.8, 91.2)
- added J4: Conn_01x02_Male, Connector_PinHeader_2.54mm:PinHeader_1x02_P2.54mm_Vertical, F.Cu at (159.8, 82.1)
- added J5: Conn_01x02_Male, Connector_PinHeader_2.54mm:PinHeader_1x02_P2.54mm_Vertical, F.Cu at (160.0, 74.4)
- added REF1: MountingHole_3.2mm_M3_ISO7380_Pad, MountingHole:MountingHole_3.2mm_M3_ISO7380_Pad, F.Cu at (98.0, 42.0)
- added REF2: MountingHole_3.2mm_M3_ISO7380_Pad, MountingHole:MountingHole_3.2mm_M3_ISO7380_Pad, F.Cu at (98.0, 111.8)
- added REF3: MountingHole_3.2mm_M3_ISO7380_Pad, MountingHole:MountingHole_3.2mm_M3_ISO7380_Pad, F.Cu at (212.0, 111.8)
- added REF4: MountingHole_3.2mm_M3_ISO7380_Pad, MountingHole:MountingHole_3.2mm_M3_ISO7380_Pad, F.Cu at (212.0, 42.0)
- Q1: value DMG2301L -> DMG2305UX
- R10: value 10K -> 1K
- R11: value 8.2K -> 20K
- R12: value 36K -> 20K
- U2: footprint Library:MAX98357 -> Package_DFN_QFN:TQFN-16-1EP_3x3mm_P0.5mm_EP1.6x1.6mm
- U3: footprint Library:BQ25172 -> Package_SON:WSON-8-1EP_2x2mm_P0.5mm_EP0.9x1.6mm
- U5: footprint Library:74HC4051 -> Package_SO:SOIC-16_3.9x9.9mm_P1.27mm
- U6: footprint Library:CD4072BM96 -> Package_SO:SOIC-14_3.9x8.7mm_P1.27mm
- moved J1 3.10 mm to (165.9, 42.5)
- moved C6 2.74 mm to (104.8, 45.2)
- moved C5 2.68 mm to (104.8, 43.2)
- moved SW5 2.52 mm to (193.6, 100.3)
- moved SW1 2.48 mm to (135.0, 100.3)
- moved SW4 2.46 mm to (174.1, 100.3)
- moved SW2 2.36 mm to (154.5, 100.3)
- moved Q1 1.37 mm to (167.1, 53.8)
- moved BT1 1.24 mm to (200.2, 44.0)
- moved U5 0.33 mm to (112.9, 78.3)
Connections:
- C7 pad 1: /Power2/USB_VBUS -> Net-(C7-Pad1)
- Q1 pad 1: /Power2/USB_VBUS -> Net-(C7-Pad1)
- R10 pad 1: /Power2/USB_VBUS -> Net-(C7-Pad1)
- U1 pad 13: unconnected-(U1-Pad13) -> GND
- U1 pad 18: unconnected-(U1-Pad18) -> GND
- U1 pad 21: unconnected-(U1-Pad21) -> Net-(J3-Pad6)
- U1 pad 22: unconnected-(U1-Pad22) -> Net-(J3-Pad5)
- U1 pad 23: unconnected-(U1-Pad23) -> GND
- U1 pad 24: unconnected-(U1-Pad24) -> Net-(J3-Pad4)
- U1 pad 25: unconnected-(U1-Pad25) -> Net-(J3-Pad3)
- U1 pad 26: unconnected-(U1-Pad26) -> Net-(J3-Pad2)
- U1 pad 28: unconnected-(U1-Pad28) -> GND
- U1 pad 3: unconnected-(U1-Pad3) -> GND
- U1 pad 33: unconnected-(U1-Pad33) -> GND
- U1 pad 38: unconnected-(U1-Pad38) -> GND
- U1 pad 8: unconnected-(U1-Pad8) -> GND
- U2 pad 4: Net-(R1-Pad2) -> VDD
- U3 pad 1: /Power2/USB_VBUS -> Net-(C7-Pad1)
Routing:
- net Net-(C7-Pad1): track 0.00 -> 65.8 mm, vias 0 -> 4
- net GND: track 32.3 -> 80.5 mm, vias 36 -> 28
- net VDD: track 10.3 -> 51.5 mm, vias 0 -> 8
- net +3.3V: track 135.6 -> 162.3 mm, vias 20 -> 18
- net Net-(J3-Pad2): track 0.00 -> 22.6 mm
- net Net-(J3-Pad3): track 0.00 -> 19.0 mm
- net Net-(J3-Pad4): track 0.00 -> 15.4 mm
- net /Power2/USB_VBUS: track 64.4 -> 79.5 mm
- net Net-(J3-Pad5): track 0.00 -> 10.5 mm
- net Net-(J3-Pad6): track 0.00 -> 6.93 mm
- net B0: track 63.4 -> 70.2 mm
- net B1: track 99.7 -> 105.8 mm
- net Net-(Q1-Pad2): track 27.4 -> 22.0 mm
- net B2: track 81.5 -> 86.8 mm
- net B3: track 118.7 -> 123.5 mm
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Other:
- board size 108.2 x 77.1 mm -> 122 x 77.8 mm
- board text added: "+"
- board text added: "-"
- board text added: "16,17,18,19,20,GND"
- board text added: "3 Cell NiMH AA"
- board text added: "AMP - BCLK: 26, LRCLK: 27, DIN: 28"
- board text added: "B0"
- board text added: "B1"
- board text added: "B2"
- board text added: "B3"
- board text added: "BAT+"
- board text added: "BAT_EN"
- board text added: "CHG_EN"
- board text added: "Gigi"
- board text added: "Input - A: 15, S0: 12, S1: 13, S2: 14"
- board text added: "MUTE"
- board text added: "OUT"
- board text added: "PICO"
- board text added: "SD - MISO: 6, CS: 7, CLK: 9, MOSI: 10"
- board text added: "V0.1 Evaluation"
- board text added: "VOL"
- board text added: "Zorro"

Commit message: update
Parts:
- added C12: 220pF, Capacitor_SMD:C_0805_2012Metric, F.Cu at (182.7, 92.8)
- added C9: 10uF, Capacitor_SMD:C_0805_2012Metric, F.Cu at (173.8, 88.9)
- added J6: Conn_01x02_Male, Connector_PinHeader_2.54mm:PinHeader_1x02_P2.54mm_Vertical, F.Cu at (181.3, 60.6)
- added J7: Screw_Terminal_Speaker, TerminalBlock:TerminalBlock_bornier-2_P5.08mm, F.Cu at (178.7, 134.7)
- added JP1: Boost EN Connect, Jumper:SolderJumper-2_P1.3mm_Bridged_RoundedPad1.0x1.5mm, F.Cu at (173.4, 74.5)
- added L1: 2.2uH, Inductor_SMD:L_Sunlord_MWSA06xxS, F.Cu at (180.2, 74.6)
- added R1: 47K, Resistor_SMD:R_0805_2012Metric, F.Cu at (189.3, 55.5)
- added R13: 10K, Resistor_SMD:R_0805_2012Metric, F.Cu at (107.0, 72.3)
- added R24: 10K, Resistor_SMD:R_0805_2012Metric, F.Cu at (186.4, 82.6)
- added REF5: MountingHole_3.2mm_M3_ISO7380_Pad, MountingHole:MountingHole_3.2mm_M3_ISO7380_Pad, F.Cu at (137.0, 47.0)
- added REF6: MountingHole_3.2mm_M3_ISO7380_Pad, MountingHole:MountingHole_3.2mm_M3_ISO7380_Pad, F.Cu at (191.0, 47.0)
- added REF7: MountingHole_3.2mm_M3_ISO7380_Pad, MountingHole:MountingHole_3.2mm_M3_ISO7380_Pad, F.Cu at (137.0, 136.0)
- added REF8: MountingHole_3.2mm_M3_ISO7380_Pad, MountingHole:MountingHole_3.2mm_M3_ISO7380_Pad, F.Cu at (191.0, 136.0)
- added U4: BQ25172, Package_SON:WSON-8-1EP_2x2mm_P0.5mm_EP0.9x1.6mm, F.Cu at (183.0, 66.8)
- added mouse-bite-2mm-slot: VAL1, Library:mouse-bite-2mm-slot, F.Cu at (132.0, 90.0)
- added mouse-bite-2mm-slot: VAL2, Library:mouse-bite-2mm-slot, F.Cu at (132.0, 53.0)
- added mouse-bite-2mm-slot: VAL3, Library:mouse-bite-2mm-slot, F.Cu at (132.0, 130.0)
- BT1: footprint Battery:BatteryHolder_Keystone_2479_3xAAA -> Battery:BatteryHolder_Keystone_2462_2xAA
- C11: value 0.1uF -> 220pF
- C3, C4: value 220pF -> 0.1uF
- C6: value 0.1uF -> 10uF
- C8: value 10uF -> 22uF
- J1: value Screw_Terminal_Speaker -> Micro_SD_Card_Det; footprint TerminalBlock:TerminalBlock_bornier-2_P5.08mm -> Connector_Card:microSD_HC_Molex_104031-0811
- J2: value Micro_SD_Card_Det -> Conn_01x06; footprint Connector_Card:microSD_HC_Molex_104031-0811 -> Connector_PinHeader_2.54mm:PinHeader_1x06_P2.54mm_Vertical
- J3: value Conn_01x06 -> Conn_01x06_Male; footprint Connector_PinHeader_2.54mm:PinHeader_1x06_P2.54mm_Vertical -> Connector_JST:JST_PH_B6B-PH-SM4-TB_1x06-1MP_P2.00mm_Vertical
- J4: value Conn_01x02_Male -> Conn_01x06_Male; footprint Connector_PinHeader_2.54mm:PinHeader_1x02_P2.54mm_Vertical -> Connector_JST:JST_PH_B6B-PH-SM4-TB_1x06-1MP_P2.00mm_Vertical
- R10: value 1K -> 10K
- R11, R12: value 20K -> 10K
- R14, R15, R16: value 2K7 -> 10K
- R17, R19: value 10K -> 1K
- R20, R21: value 10K -> 20K
- R23: value 10K -> 90.9K
- R7: value 47K -> 2K7
- R8: value 1K -> 2K7
- R9: value 10K -> 2K7
- SW1, SW2, SW3, SW4, SW5: moved to B.Cu
- U2: value MAX98357 -> 74HC4051; footprint Package_DFN_QFN:TQFN-16-1EP_3x3mm_P0.5mm_EP1.6x1.6mm -> Package_SO:SOIC-16_3.9x9.9mm_P1.27mm
- U3: value BQ25172 -> 4072; footprint Package_SON:WSON-8-1EP_2x2mm_P0.5mm_EP0.9x1.6mm -> Package_SO:SOIC-14_3.9x8.7mm_P1.27mm
- U5: value 74HC4051 -> TLV61070A; footprint Package_SO:SOIC-16_3.9x9.9mm_P1.27mm -> Package_SO:TSOP-6_1.65x3.05mm_P0.95mm
- U6: value 4072 -> MAX98357; footprint Package_SO:SOIC-14_3.9x8.7mm_P1.27mm -> Package_DFN_QFN:TQFN-16-1EP_3x3mm_P0.5mm_EP1.6x1.6mm
- moved REF4 126.7 mm to (127.0, 136.0)
- moved REF3 108.7 mm to (106.0, 136.0)
- moved R20 89.5 mm to (189.6, 65.2), turned to 90 degrees
- moved R21 85.4 mm to (187.6, 65.2), turned to 90 degrees
- moved C6 82.2 mm to (184.8, 64.4)
- moved R19 80.6 mm to (186.6, 70.4), turned to 0 degrees
- moved C5 79.2 mm to (181.2, 64.5), turned to 0 degrees
- moved BT1 77.2 mm to (191.4, 120.8), turned to 180 degrees
- moved SW5 75.8 mm to (122.0, 125.2), turned to 90 degrees
- moved C4 72.2 mm to (113.9, 104.7), turned to -90 degrees
- moved REF2 71.0 mm to (127.0, 47.0)
- moved R17 70.8 mm to (179.9, 68.1), turned to 90 degrees
- moved U6 69.9 mm to (179.2, 89.0)
- moved U5 69.5 mm to (182.3, 82.5)
- moved C3 68.4 mm to (113.5, 92.0), turned to 90 degrees
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Connections:
- C1 pad 1: VDD -> +3.3V
- C10 pad 1: +3.3V -> VDD
- C11 pad 1: +3.3V -> Net-(C11-Pad1)
- C2 pad 1: VDD -> +3.3V
- C3 pad 1: Net-(C3-Pad1) -> /Input/3.3V_LOCAL
- C3 pad 2: GND -> /Input/GND_LOCAL
- C4 pad 1: GND -> /Input/3.3V_LOCAL
- C4 pad 2: Net-(C4-Pad2) -> /Input/GND_LOCAL
- C5 pad 1: +3.3V -> Net-(C5-Pad1)
- C6 pad 1: +3.3V -> Net-(BT1-Pad1)
- C7 pad 1: Net-(C7-Pad1) -> /Power/OUT
- C8 pad 1: Net-(BT1-Pad1) -> VDD
- FB1 pad 2: Net-(C3-Pad1) -> Net-(C11-Pad1)
- FB2 pad 2: Net-(C4-Pad2) -> Net-(C12-Pad2)
- J1 pad 1: Net-(C3-Pad1) -> Net-(J1-Pad1)
- J1 pad 2: Net-(C4-Pad2) -> SD_CS
- J2 pad 1: Net-(J2-Pad1) -> GND
- J2 pad 2: SD_CS -> GND
- J2 pad 3: SD_MOSI -> Net-(J2-Pad3)
- J2 pad 4: +3.3V -> Net-(J2-Pad4)
- J2 pad 5: SD_CLK -> Net-(J2-Pad5)
- J2 pad 6: GND -> Net-(J2-Pad6)
- J3 pad 2: Net-(J3-Pad2) -> +3.3V
- J3 pad 3: Net-(J3-Pad3) -> GP14
- J3 pad 4: Net-(J3-Pad4) -> GP13
- J3 pad 5: Net-(J3-Pad5) -> GP12
- J3 pad 6: Net-(J3-Pad6) -> GP15
- J4 pad 1: Net-(C7-Pad1) -> /Input/GND_LOCAL
- J4 pad 2: /Power2/USB_VBUS -> /Input/3.3V_LOCAL
- J5 pad 1: VDD -> Net-(C5-Pad1)
- J5 pad 2: Net-(Q1-Pad2) -> /Power/USB_VBUS
- Q1 pad 1: Net-(C7-Pad1) -> Net-(C5-Pad1)
- Q1 pad 2: Net-(Q1-Pad2) -> Net-(J6-Pad2)
- R10 pad 1: Net-(C7-Pad1) -> B0
- R10 pad 2: Net-(D1-Pad2) -> /Input/GND_LOCAL
- R11 pad 1: Net-(R11-Pad1) -> B2
- R11 pad 2: GND -> /Input/GND_LOCAL
- R12 pad 1: Net-(R12-Pad1) -> B4
- R12 pad 2: GND -> /Input/GND_LOCAL
- R14 pad 1: GP12 -> B6
- R14 pad 2: GND -> /Input/GND_LOCAL
- R15 pad 1: GP13 -> B1
- R15 pad 2: GND -> /Input/GND_LOCAL
- R16 pad 1: GP14 -> B3
- R16 pad 2: GND -> /Input/GND_LOCAL
- R17 pad 1: B0 -> GND
- R17 pad 2: GND -> Net-(R17-Pad2)
- R18 pad 1: B2 -> GND
- R18 pad 2: GND -> Net-(R18-Pad2)
- R19 pad 1: B4 -> Net-(C5-Pad1)
- R19 pad 2: GND -> Net-(D1-Pad2)
- R2 pad 2: Net-(J2-Pad8) -> SD_MISO
- R20 pad 1: B5 -> Net-(R20-Pad1)
- R21 pad 1: B6 -> Net-(R21-Pad1)
- R22 pad 1: B1 -> /Power/OUT
- R22 pad 2: GND -> Net-(JP1-Pad2)
- R23 pad 1: B3 -> VDD
- R23 pad 2: GND -> Net-(R23-Pad2)
- R3 pad 2: SD_MISO -> SD_CLK
- R4 pad 2: SD_CLK -> SD_MOSI
- R5 pad 2: SD_MOSI -> SD_CS
- R6 pad 2: SD_CS -> Net-(J1-Pad1)
- R7 pad 1: +3.3V -> /Input/S0
- R7 pad 2: Net-(J2-Pad1) -> /Input/GND_LOCAL
- R8 pad 1: GND -> /Input/S1
- R8 pad 2: Net-(R8-Pad2) -> /Input/GND_LOCAL
- R9 pad 1: GND -> /Input/S2
- R9 pad 2: Net-(R9-Pad2) -> /Input/GND_LOCAL
- SW1 pad 2: +3.3V -> /Input/3.3V_LOCAL
- SW2 pad 2: +3.3V -> /Input/3.3V_LOCAL
- SW3 pad C: +3.3V -> /Input/3.3V_LOCAL
- SW3 pad S1: +3.3V -> /Input/3.3V_LOCAL
- SW4 pad 2: +3.3V -> /Input/3.3V_LOCAL
- SW5 pad 2: +3.3V -> /Input/3.3V_LOCAL
- U1 pad 1: unconnected-(U1-Pad1) -> Net-(J2-Pad6)
- U1 pad 2: unconnected-(U1-Pad2) -> Net-(J2-Pad5)
- U1 pad 21: Net-(J3-Pad6) -> unconnected-(U1-Pad21)
- U1 pad 22: Net-(J3-Pad5) -> unconnected-(U1-Pad22)
- U1 pad 24: Net-(J3-Pad4) -> unconnected-(U1-Pad24)
- U1 pad 25: Net-(J3-Pad3) -> unconnected-(U1-Pad25)
- U1 pad 26: Net-(J3-Pad2) -> unconnected-(U1-Pad26)
- U1 pad 29: unconnected-(U1-Pad29) -> /Sound/SPEAKER_EN
- U1 pad 39: VDD -> /Power/OUT
- U1 pad 4: unconnected-(U1-Pad4) -> Net-(J2-Pad4)
- U1 pad 40: /Power2/USB_VBUS -> /Power/USB_VBUS
- U1 pad 5: unconnected-(U1-Pad5) -> Net-(J2-Pad3)
- U2 pad 1: GP28 -> B3
- U2 pad 10: Net-(FB2-Pad1) -> /Input/S1
- U2 pad 11: GND -> /Input/S0
- U2 pad 12: (no net) -> B2
- U2 pad 13: (no net) -> ANY
- U2 pad 14: GP27 -> B0
- U2 pad 15: GND -> B1
- U2 pad 16: GP26 -> /Input/3.3V_LOCAL
- U2 pad 2: VDD -> B5
- U2 pad 3: GND -> /Input/A
- U2 pad 4: VDD -> B6
- U2 pad 5: (no net) -> B4
- U2 pad 6: (no net) -> /Input/GND_LOCAL
- U2 pad 7: VDD -> /Input/GND_LOCAL
- U2 pad 8: VDD -> /Input/GND_LOCAL
- U2 pad 9: Net-(FB1-Pad1) -> /Input/S2
- U3 pad 1: Net-(C7-Pad1) -> Net-(U3-Pad1)
- U3 pad 2: Net-(R8-Pad2) -> B0
- U3 pad 3: Net-(R9-Pad2) -> B1
- U3 pad 4: GND -> B2
- U3 pad 5: Net-(D1-Pad1) -> B3
- U3 pad 6: Net-(R11-Pad1) -> (no net)
- U3 pad 7: Net-(R12-Pad1) -> /Input/GND_LOCAL
- U3 pad 8: Net-(BT1-Pad1) -> (no net)
- U3 pad 9: GND -> Net-(U3-Pad1)
- U5 pad 1: B3 -> Net-(L1-Pad2)
- U5 pad 2: B5 -> GND
- U5 pad 3: GP15 -> Net-(JP1-Pad2)
- U5 pad 4: B6 -> Net-(R23-Pad2)
- U5 pad 5: B4 -> VDD
- U5 pad 6: GND -> /Power/OUT
- U6 pad 1: Net-(U6-Pad1) -> GP28
- U6 pad 10: B4 -> Net-(FB2-Pad1)
- U6 pad 11: B5 -> GND
- U6 pad 12: B6 -> (no net)
- U6 pad 13: ANY -> (no net)
- U6 pad 14: +3.3V -> GP27
- U6 pad 2: B0 -> VDD
- U6 pad 3: B1 -> GND
- U6 pad 4: B2 -> VDD
- U6 pad 5: B3 -> (no net)
- U6 pad 7: GND -> VDD
- U6 pad 8: (no net) -> VDD
- U6 pad 9: Net-(U6-Pad1) -> Net-(FB1-Pad1)
Routing:
- net /Power/OUT: track 0.00 -> 82.3 mm, vias 0 -> 2
- net /Power2/USB_VBUS: track 79.5 -> 0.00 mm, vias 2 -> 0
- net Net-(C7-Pad1): track 65.8 -> 0.00 mm, vias 4 -> 0
- net /Input/S1: track 0.00 -> 53.0 mm, vias 0 -> 2
- net /Input/GND_LOCAL: track 0.00 -> 51.1 mm, vias 0 -> 10
- net B1: track 105.8 -> 58.2 mm, vias 4 -> 0
- net B3: track 123.5 -> 78.3 mm, vias 3 -> 2
- net +3.3V: track 162.3 -> 117.8 mm, vias 18 -> 4
- net Net-(C11-Pad1): track 0.00 -> 43.4 mm
- net Net-(C12-Pad2): track 0.00 -> 43.2 mm
- net /Input/S2: track 0.00 -> 41.7 mm, vias 0 -> 2
- net B5: track 52.1 -> 93.6 mm, vias 0 -> 4
- net /Input/3.3V_LOCAL: track 0.00 -> 40.1 mm, vias 0 -> 8
- net Net-(C5-Pad1): track 0.00 -> 39.1 mm, vias 0 -> 2
- net /Input/S0: track 0.00 -> 30.2 mm, vias 0 -> 2
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- added copper zone on F.Cu, net /Input/3.3V_LOCAL
- added copper zone on B.Cu, net /Input/GND_LOCAL
- removed copper zone on F.Cu, net +3.3V
- removed copper zone on F.Cu, net VDD
Other:
- board size 122 x 77.8 mm -> 93 x 97 mm
- board text added: "2 Cell NiMH AA"
- board text added: "PLACE OTHER SIDE"
- board text removed: "16,17,18,19,20,GND"
- board text removed: "3 Cell NiMH AA"
- board text removed: "Gigi"
- board text removed: "OUT"
- board text removed: "PICO"
- board text removed: "Zorro"

Commit message: update
Parts:
- added J8: Conn_01x02_Male, Connector_PinHeader_2.54mm:PinHeader_1x02_P2.54mm_Vertical, F.Cu at (184.5, 89.5)
Connections:
- C8 pad 1: VDD -> /Sound/V_BOOST
- R23 pad 1: VDD -> /Sound/V_BOOST
- U5 pad 5: VDD -> /Sound/V_BOOST
Routing:
- net /Sound/V_BOOST: track 0.00 -> 21.9 mm
- net VDD: track 33.4 -> 17.9 mm
Other:
- board text added: "BAT_AUD_EN"
- board text added: "BOOST_EN"
- board text added: "TO_AUD"
- board text added: "VOL/MUTE"
- board text removed: "MUTE"
- board text removed: "VOL"

Commit message: update, schematic should be done
Parts:
- removed J8: Conn_01x02_Male, Connector_PinHeader_2.54mm:PinHeader_1x02_P2.54mm_Vertical
- removed JP1: Boost EN Connect, Jumper:SolderJumper-2_P1.3mm_Bridged_RoundedPad1.0x1.5mm
- removed R21: 20K, Resistor_SMD:R_0805_2012Metric
- removed R22, R24: 10K, Resistor_SMD:R_0805_2012Metric
- removed R23: 90.9K, Resistor_SMD:R_0805_2012Metric
- removed REF1, REF2, REF3, REF4, REF5, REF6, REF7, REF8: MountingHole_3.2mm_M3_ISO7380_Pad, MountingHole:MountingHole_3.2mm_M3_ISO7380_Pad
- removed mouse-bite-2mm-slot: VAL1, Library:mouse-bite-2mm-slot
- removed mouse-bite-2mm-slot: VAL2, Library:mouse-bite-2mm-slot
- removed mouse-bite-2mm-slot: VAL3, Library:mouse-bite-2mm-slot
- added C13: 220pF, Capacitor_SMD:C_0805_2012Metric, F.Cu at (156.8, 103.0)
- added C14: 27pF, Capacitor_SMD:C_0603_1608Metric, F.Cu at (173.7, 66.3)
- added C15: 27pF, Capacitor_SMD:C_0603_1608Metric, F.Cu at (184.1, 54.5)
- added C16: 100nF, Capacitor_SMD:C_0603_1608Metric, F.Cu at (184.1, 57.0)
- added C17: 100nF, Capacitor_SMD:C_0603_1608Metric, F.Cu at (168.4, 73.0)
- added C18: 1uF, Capacitor_SMD:C_0603_1608Metric, F.Cu at (178.0, 63.8)
- added C19: 100nF, Capacitor_SMD:C_0603_1608Metric, F.Cu at (188.1, 52.0)
- added C20: 1uF, Capacitor_SMD:C_0603_1608Metric, F.Cu at (169.7, 68.0)
- added C21: 100nF, Capacitor_SMD:C_0603_1608Metric, F.Cu at (184.1, 52.0)
- added C22: 100nF, Capacitor_SMD:C_0603_1608Metric, F.Cu at (174.0, 61.3)
- added C23: 100nF, Capacitor_SMD:C_0603_1608Metric, F.Cu at (168.4, 70.5)
- added C24: 100nF, Capacitor_SMD:C_0603_1608Metric, F.Cu at (164.4, 70.0)
- added C25: 100nF, Capacitor_SMD:C_0603_1608Metric, F.Cu at (164.5, 72.1)
- added C26: 100nF, Capacitor_SMD:C_0603_1608Metric, F.Cu at (174.0, 63.8)
- added C27: 100nF, Capacitor_SMD:C_0603_1608Metric, F.Cu at (182.0, 61.3)
- added D2: DF2S6.8FS, Diode_SMD:D_SOD-923, F.Cu at (232.7, 107.8)
- added D3: DF2S6.8FS, Diode_SMD:D_SOD-923, F.Cu at (251.7, 88.2)
- added D4: B5819W SL, Diode_SMD:D_SOD-123, F.Cu at (90.3, 86.9)
- added D5: CHARGE_LED, LED_SMD:LED_0805_2012Metric, F.Cu at (98.7, 91.2)
- added H1: MountingHole, MountingHole:MountingHole_3.2mm_M3_DIN965_Pad, F.Cu at (217.4, 29.8)
- added H2: MountingHole, MountingHole:MountingHole_3.2mm_M3_DIN965_Pad, F.Cu at (59.2, 67.5)
- added H3: MountingHole, MountingHole:MountingHole_3.2mm_M3_DIN965_Pad, F.Cu at (224.5, 37.0)
- added H4: MountingHole, MountingHole:MountingHole_3.2mm_M3_DIN965_Pad, F.Cu at (224.5, 29.8)
- added SW6: BOOTSEL, Button_Switch_SMD:SW_SPST_SKQG_WithoutStem, F.Cu at (167.2, 60.9)
- added U7: W25Q128JVS, Package_SO:SOIC-8_5.23x5.23mm_P1.27mm, F.Cu at (167.6, 54.1)
- added Y1: X322512MSB4SI, Crystal:Crystal_SMD_3225-4Pin_3.2x2.5mm, F.Cu at (165.0, 66.4)
- C10, C4: value 0.1uF -> 10uF
- C11: value 220pF -> 0.1uF
- C6: value 10uF -> 22uF
- C8: value 22uF -> 10uF
- D1: value CHARGE_LED -> DF2S6.8FS; footprint LED_SMD:LED_0805_2012Metric -> Diode_SMD:D_SOD-923
- J1: value Micro_SD_Card_Det -> USB_C_Receptacle_USB2.0; footprint Connector_Card:microSD_HC_Molex_104031-0811 -> Connector_USB:USB_C_Receptacle_G-Switch_GT-USB-7010ASV
- J3: value Conn_01x06_Male -> Micro_SD_Card_Det; footprint Connector_JST:JST_PH_B6B-PH-SM4-TB_1x06-1MP_P2.00mm_Vertical -> Connector_Card:microSD_HC_Molex_104031-0811
- J4: value Conn_01x06_Male -> Conn_01x05_Male; footprint Connector_JST:JST_PH_B6B-PH-SM4-TB_1x06-1MP_P2.00mm_Vertical -> Connector_JST:JST_PH_B5B-PH-SM4-TB_1x05-1MP_P2.00mm_Vertical
- J5: value Conn_01x02_Male -> Conn_01x05_Male; footprint Connector_PinHeader_2.54mm:PinHeader_1x02_P2.54mm_Vertical -> Connector_JST:JST_PH_B5B-PH-SM4-TB_1x05-1MP_P2.00mm_Vertical
- J6: value Conn_01x02_Male -> PWR_EN
- L1: footprint Inductor_SMD:L_Sunlord_MWSA06xxS -> Inductor_SMD:L_Sunlord_MWSA05xxS
- R1, R2: value 47K -> 5.1K
- R10: value 10K -> 27R
- R11, R18: value 10K -> 1K; footprint Resistor_SMD:R_0805_2012Metric -> Resistor_SMD:R_0603_1608Metric
- R12, R19: footprint Resistor_SMD:R_0805_2012Metric -> Resistor_SMD:R_0603_1608Metric
- R13, R15: value 10K -> 2K7
- R14: value 10K -> 24.3K
- R16: value 10K -> 27K
- R17: value 1K -> 20K
- R20: value 20K -> 10K; footprint Resistor_SMD:R_0805_2012Metric -> Resistor_SMD:R_0603_1608Metric
- R3, R4, R5, R6: value 47K -> 10K; footprint Resistor_SMD:R_0805_2012Metric -> Resistor_SMD:R_0603_1608Metric
- R7, R8: value 2K7 -> 10K; footprint Resistor_SMD:R_0805_2012Metric -> Resistor_SMD:R_0603_1608Metric
- R9: value 2K7 -> 27R
- SW1, SW2, SW4, SW5: footprint Button_Switch_Keyboard:SW_Cherry_MX_1.00u_PCB -> Library:Kailh_socket_MX; moved to F.Cu
- SW3: moved to F.Cu
- U1: value Pico -> MCP23017_ML; footprint Library:RPI_PICO_smd -> Package_DFN_QFN:QFN-28-1EP_6x6mm_P0.65mm_EP4.25x4.25mm
- U2: value 74HC4051 -> BQ25172; footprint Package_SO:SOIC-16_3.9x9.9mm_P1.27mm -> Package_SON:WSON-8-1EP_2x2mm_P0.5mm_EP0.9x1.6mm
- U3: value 4072 -> TLV61070A; footprint Package_SO:SOIC-14_3.9x8.7mm_P1.27mm -> Package_SO:TSOP-6_1.65x3.05mm_P0.95mm
- U4: value BQ25172 -> XC6206P332MR; footprint Package_SON:WSON-8-1EP_2x2mm_P0.5mm_EP0.9x1.6mm -> Package_TO_SOT_SMD:SOT-23-3
- U5: value TLV61070A -> MAX98357; footprint Package_SO:TSOP-6_1.65x3.05mm_P0.95mm -> Package_DFN_QFN:TQFN-16-1EP_3x3mm_P0.5mm_EP1.6x1.6mm
- U6: value MAX98357 -> RP2040; footprint Package_DFN_QFN:TQFN-16-1EP_3x3mm_P0.5mm_EP1.6x1.6mm -> Package_DFN_QFN:QFN-56-1EP_7x7mm_P0.4mm_EP3.2x3.2mm
- moved R8 131.8 mm to (248.3, 91.5), turned to 0 degrees
- moved R7 130.7 mm to (243.5, 98.0), turned to 0 degrees
- moved J4 125.8 mm to (233.7, 92.5), turned to 0 degrees
- moved R9 124.5 mm to (244.1, 91.7), turned to 0 degrees
- moved J1 121.7 mm to (59.0, 42.0), turned to 90 degrees
- moved R4 108.7 mm to (248.3, 88.5)
- moved R3 106.3 mm to (243.9, 94.4)
- moved R2 105.8 mm to (239.3, 98.2)
- moved C5 103.2 mm to (82.2, 93.5)
- moved R5 101.0 mm to (228.9, 111.1)
- moved R10 99.5 mm to (224.7, 111.3)
- moved L1 97.5 mm to (83.7, 88.6), turned to 0 degrees
- moved Q1 96.4 mm to (95.7, 87.5), turned to 0 degrees
- moved U1 91.4 mm to (84.0, 120.2)
- moved BT1 88.9 mm to (124.7, 62.0)
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Connections:
- C11 pad 1: Net-(C11-Pad1) -> VDD
- C12 pad 1: GND -> Net-(C12-Pad1)
- C12 pad 2: Net-(C12-Pad2) -> GND
- C4 pad 1: /Input/3.3V_LOCAL -> Net-(C4-Pad1)
- C4 pad 2: /Input/GND_LOCAL -> GND
- C5 pad 1: Net-(C5-Pad1) -> /Power/BAT_OR_USB_POWER
- C6 pad 1: Net-(BT1-Pad1) -> VDD
- C7 pad 1: /Power/OUT -> Net-(BT1-Pad1)
- C8 pad 1: /Sound/V_BOOST -> VDD
- C9 pad 1: VDD -> +3.3V
- D1 pad 1: Net-(D1-Pad1) -> /USB_VBUS
- D1 pad 2: Net-(D1-Pad2) -> GND
- FB1 pad 2: Net-(C11-Pad1) -> Net-(C12-Pad1)
- FB2 pad 2: Net-(C12-Pad2) -> Net-(C13-Pad2)
- J2 pad 1: GND -> /rp2040/GPIO16
- J2 pad 2: GND -> /rp2040/GPIO17
- J2 pad 3: Net-(J2-Pad3) -> /rp2040/GPIO18
- J2 pad 4: Net-(J2-Pad4) -> /rp2040/GPIO19
- J2 pad 5: Net-(J2-Pad5) -> /rp2040/GPIO20
- J2 pad 6: Net-(J2-Pad6) -> /rp2040/GPIO21
- J3 pad 1: GND -> SD_DAT2
- J3 pad 2: +3.3V -> SD_CS
- J3 pad 3: GP14 -> SD_MOSI
- J3 pad 4: GP13 -> +3.3V
- J3 pad 5: GP12 -> SD_CLK
- J3 pad 6: GP15 -> GND
- J4 pad 1: /Input/GND_LOCAL -> GND
- J4 pad 2: /Input/3.3V_LOCAL -> +3.3V
- J4 pad 3: /Input/S2 -> INT
- J4 pad 4: /Input/S1 -> RP2040_SDA
- J4 pad 5: /Input/S0 -> RP2040_SCL
- J5 pad 1: Net-(C5-Pad1) -> /Input/GND_LOCAL
- J5 pad 2: /Power/USB_VBUS -> /Input/3.3V_LOCAL
- J6 pad 1: /Power/OUT -> /Power/BAT_OR_USB_POWER
- J7 pad 1: Net-(C11-Pad1) -> Net-(C12-Pad1)
- J7 pad 2: Net-(C12-Pad2) -> Net-(C13-Pad2)
- L1 pad 1: /Power/OUT -> /Power/BAT_OR_USB_POWER
- Q1 pad 1: Net-(C5-Pad1) -> Net-(C4-Pad1)
- R1 pad 1: +3.3V -> GND
- R1 pad 2: Net-(J1-Pad8) -> Net-(J1-PadB5)
- R10 pad 1: B0 -> Net-(D3-Pad1)
- R10 pad 2: /Input/GND_LOCAL -> /USB_D-
- R11 pad 1: B2 -> GND
- R11 pad 2: /Input/GND_LOCAL -> Net-(R11-Pad2)
- R12 pad 1: B4 -> GND
- R12 pad 2: /Input/GND_LOCAL -> Net-(R12-Pad2)
- R13 pad 1: B5 -> Net-(C4-Pad1)
- R13 pad 2: /Input/GND_LOCAL -> Net-(D5-Pad2)
- R14 pad 1: B6 -> VDD
- R14 pad 2: /Input/GND_LOCAL -> Net-(R14-Pad2)
- R15 pad 1: B1 -> Net-(R14-Pad2)
- R15 pad 2: /Input/GND_LOCAL -> GND
- R16 pad 1: B3 -> Net-(R16-Pad1)
- R16 pad 2: /Input/GND_LOCAL -> GND
- R17 pad 1: GND -> Net-(R17-Pad1)
- R17 pad 2: Net-(R17-Pad2) -> GND
- R18 pad 1: GND -> Net-(C15-Pad1)
- R19 pad 1: Net-(C5-Pad1) -> /rp2040/~{USB_BOOT}
- R19 pad 2: Net-(D1-Pad2) -> /rp2040/QSPI_SS
- R2 pad 1: +3.3V -> Net-(J1-PadA5)
- R2 pad 2: SD_MISO -> GND
- R20 pad 1: Net-(R20-Pad1) -> +3.3V
- R20 pad 2: GND -> /rp2040/QSPI_SS
- R3 pad 2: SD_CLK -> SD_DAT1
- R4 pad 2: SD_MOSI -> SD_MISO
- R5 pad 1: +3.3V -> SD_CLK
- R5 pad 2: SD_CS -> GND
- R6 pad 2: Net-(J1-Pad1) -> SD_MOSI
- R7 pad 1: /Input/S0 -> +3.3V
- R7 pad 2: /Input/GND_LOCAL -> SD_CS
- R8 pad 1: /Input/S1 -> +3.3V
- R8 pad 2: /Input/GND_LOCAL -> SD_DAT2
- R9 pad 1: /Input/S2 -> Net-(D2-Pad1)
- R9 pad 2: /Input/GND_LOCAL -> /USB_D+
- SW1 pad 2: /Input/3.3V_LOCAL -> /Input/GND_LOCAL
- SW2 pad 1: B2 -> B1
- SW2 pad 2: /Input/3.3V_LOCAL -> /Input/GND_LOCAL
- SW3 pad C: /Input/3.3V_LOCAL -> /Input/GND_LOCAL
- SW3 pad S1: /Input/3.3V_LOCAL -> /Input/GND_LOCAL
- SW4 pad 1: B1 -> B2
- SW4 pad 2: /Input/3.3V_LOCAL -> /Input/GND_LOCAL
- SW5 pad 2: /Input/3.3V_LOCAL -> /Input/GND_LOCAL
- U1 pad 1: Net-(J2-Pad6) -> B4
- U1 pad 10: SD_MOSI -> unconnected-(U1-Pad10)
- U1 pad 11: unconnected-(U1-Pad11) -> /Input/GND_LOCAL
- U1 pad 12: unconnected-(U1-Pad12) -> /Input/GND_LOCAL
- U1 pad 13: GND -> /Input/GND_LOCAL
- U1 pad 14: unconnected-(U1-Pad14) -> /Input/3.3V_LOCAL
- U1 pad 15: unconnected-(U1-Pad15) -> /Input/INT
- U1 pad 16: GP12 -> unconnected-(U1-Pad16)
- U1 pad 17: GP13 -> unconnected-(U1-Pad17)
- U1 pad 18: GND -> unconnected-(U1-Pad18)
- U1 pad 19: GP14 -> unconnected-(U1-Pad19)
- U1 pad 2: Net-(J2-Pad5) -> B5
- U1 pad 20: GP15 -> unconnected-(U1-Pad20)
- U1 pad 23: GND -> unconnected-(U1-Pad23)
- U1 pad 25: unconnected-(U1-Pad25) -> B0
- U1 pad 26: unconnected-(U1-Pad26) -> B1
- U1 pad 27: unconnected-(U1-Pad27) -> B2
- U1 pad 28: GND -> B3
- U1 pad 29: /Sound/SPEAKER_EN -> /Input/GND_LOCAL
- U1 pad 3: GND -> B6
- U1 pad 4: Net-(J2-Pad4) -> unconnected-(U1-Pad4)
- U1 pad 5: Net-(J2-Pad3) -> /Input/3.3V_LOCAL
- U1 pad 6: SD_MISO -> /Input/GND_LOCAL
- U1 pad 7: SD_CS -> unconnected-(U1-Pad7)
- U1 pad 8: GND -> /Input/SCK
- U1 pad 9: SD_CLK -> /Input/SDA
- U2 pad 1: B3 -> Net-(C4-Pad1)
- U2 pad 2: B5 -> Net-(R11-Pad2)
- U2 pad 3: /Input/A -> Net-(R12-Pad2)
- U2 pad 4: B6 -> GND
- U2 pad 5: B4 -> Net-(D5-Pad1)
- U2 pad 6: /Input/GND_LOCAL -> Net-(R16-Pad1)
- U2 pad 7: /Input/GND_LOCAL -> Net-(R17-Pad1)
- U2 pad 8: /Input/GND_LOCAL -> Net-(BT1-Pad1)
- U2 pad 9: /Input/S2 -> GND
- U3 pad 1: Net-(U3-Pad1) -> Net-(L1-Pad2)
- U3 pad 2: B0 -> GND
- U3 pad 3: B1 -> /Power/BAT_OR_USB_POWER
- U3 pad 4: B2 -> Net-(R14-Pad2)
- U3 pad 5: B3 -> VDD
- U3 pad 6: (no net) -> /Power/BAT_OR_USB_POWER
- U4 pad 1: Net-(C5-Pad1) -> GND
- U4 pad 2: Net-(R17-Pad2) -> +3.3V
- U4 pad 3: Net-(R18-Pad2) -> VDD
- U5 pad 1: Net-(L1-Pad2) -> GP28
- U5 pad 2: GND -> VDD
- U5 pad 3: Net-(JP1-Pad2) -> GND
- U5 pad 4: Net-(R23-Pad2) -> VDD
- U5 pad 5: /Sound/V_BOOST -> (no net)
- U5 pad 6: /Power/OUT -> (no net)
- U6 pad 1: GP28 -> +3.3V
- U6 pad 10: Net-(FB2-Pad1) -> +3.3V
- U6 pad 11: GND -> INT
- U6 pad 12: (no net) -> /rp2040/GPIO9
- U6 pad 13: (no net) -> /rp2040/GPIO10
- U6 pad 14: GP27 -> /rp2040/GPIO11
- U6 pad 15: GND -> /rp2040/GPIO12
- U6 pad 16: GP26 -> /rp2040/GPIO13
- U6 pad 17: GND -> /rp2040/GPIO14
- U6 pad 2: VDD -> SD_MISO
- U6 pad 3: GND -> SD_CS
- U6 pad 4: VDD -> SD_CLK
- U6 pad 5: (no net) -> SD_MOSI
- U6 pad 6: (no net) -> SD_DAT1
- U6 pad 7: VDD -> SD_DAT2
- U6 pad 8: VDD -> RP2040_SDA
- U6 pad 9: Net-(FB1-Pad1) -> RP2040_SCL
Routing:
- net +3.3V: track 117.8 -> 0.00 mm, vias 4 -> 0
- net B5: track 93.6 -> 0.00 mm, vias 4 -> 0
- net /Power/OUT: track 82.3 -> 0.00 mm, vias 2 -> 0
- net GND: track 80.5 -> 0.00 mm, vias 31 -> 0
- net B3: track 78.3 -> 0.00 mm, vias 2 -> 0
- net B4: track 73.9 -> 0.00 mm
- net B2: track 72.3 -> 0.00 mm, vias 2 -> 0
- net Net-(BT1-Pad1): track 71.9 -> 0.00 mm
- net B6: track 67.7 -> 0.00 mm, vias 2 -> 0
- net B0: track 61.6 -> 0.00 mm, vias 3 -> 0
- net B1: track 58.2 -> 0.00 mm
- net SD_MOSI: track 54.5 -> 0.00 mm, vias 1 -> 0
- net /Input/S1: track 53.0 -> 0.00 mm, vias 2 -> 0
- net SD_CLK: track 51.5 -> 0.00 mm, vias 3 -> 0
- net /Input/GND_LOCAL: track 51.1 -> 0.00 mm, vias 10 -> 0
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- removed copper zone on F.Cu, net /Input/3.3V_LOCAL
- removed copper zone on B.Cu, net /Input/GND_LOCAL
- removed copper zone on B.Cu, net GND
Other:
- board size 93 x 97 mm -> 92.5 x 39.1 mm
- board text removed: "+"
- board text removed: "-"
- board text removed: "2 Cell NiMH AA"
- board text removed: "AMP - BCLK: 26, LRCLK: 27, DIN: 28"
- board text removed: "B0"
- board text removed: "B1"
- board text removed: "B2"
- board text removed: "B3"
- board text removed: "BAT+"
- board text removed: "BAT_AUD_EN"
- board text removed: "BAT_EN"
- board text removed: "BOOST_EN"
- board text removed: "CHG_EN"
- board text removed: "Input - A: 15, S0: 12, S1: 13, S2: 14"
- board text removed: "PLACE OTHER SIDE"
- board text removed: "SD - MISO: 6, CS: 7, CLK: 9, MOSI: 10"
- board text removed: "TO_AUD"
- board text removed: "V0.1 Evaluation"
- board text removed: "VOL/MUTE"

Commit message: wip
Parts:
- C1, C10, C12, C13, C4, C5, C6, C7, C8, C9: footprint Capacitor_SMD:C_0805_2012Metric -> Capacitor_SMD:C_0603_1608Metric
- C11, C2, C3: value 0.1uF -> 100nF; footprint Capacitor_SMD:C_0805_2012Metric -> Capacitor_SMD:C_0603_1608Metric
- R1, R13, R15, R16, R17, R2: footprint Resistor_SMD:R_0805_2012Metric -> Resistor_SMD:R_0603_1608Metric
- moved H2 224.6 mm to (282.1, 94.3)
- moved R4 206.6 mm to (73.7, -21.8)
- moved R8 204.8 mm to (77.7, -21.8)
- moved R6 203.3 mm to (75.3, -19.3)
- moved R7 198.6 mm to (81.7, -17.1)
- moved R5 198.3 mm to (81.5, -21.6)
- moved C2 197.1 mm to (77.7, -16.8)
- moved C1 196.2 mm to (73.7, -16.8)
- moved R3 195.1 mm to (86.1, -20.3)
- moved C12 194.5 mm to (111.9, -77.3)
- moved J5 193.7 mm to (25.3, 152.6)
- moved FB1 192.9 mm to (112.1, -80.1)
- moved C5 188.1 mm to (212.8, -41.8)
- moved C13 187.7 mm to (116.3, -80.3)
- moved BT1 187.0 mm to (207.5, -105.7), turned to 0 degrees
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Connections:
- J2 pad 1: /rp2040/GPIO16 -> /rp2040/GPIO12
- J2 pad 2: /rp2040/GPIO17 -> /rp2040/GPIO13
- J2 pad 3: /rp2040/GPIO18 -> /rp2040/GPIO14
- J2 pad 4: /rp2040/GPIO19 -> /rp2040/GPIO15
- J2 pad 5: /rp2040/GPIO20 -> /rp2040/GPIO16
- J2 pad 6: /rp2040/GPIO21 -> /rp2040/GPIO17
- U5 pad 1: GP28 -> AMP_DIN
- U5 pad 14: GP27 -> AMP_LRCLK
- U5 pad 16: GP26 -> AMP_BCLK
- U6 pad 12: /rp2040/GPIO9 -> AMP_BCLK
- U6 pad 13: /rp2040/GPIO10 -> AMP_LRCLK
- U6 pad 14: /rp2040/GPIO11 -> AMP_DIN
- U6 pad 38: GP26 -> /rp2040/GPIO26_ADC0
- U6 pad 39: GP27 -> /rp2040/GPIO27_ADC1
- U6 pad 40: GP28 -> /rp2040/GPIO28_ADC2
Other:
- board outline removed

Commit message: update
Parts:
- BT1, SW1, SW2, SW4, SW5: moved to B.Cu
- C11, C16, C17, C18, C19, C2, C20, C21, C22, C23, C24, C25, C26, C27, C3: footprint Capacitor_SMD:C_0603_1608Metric -> Capacitor_SMD:C_0402_1005Metric
- R10, R9: footprint Resistor_SMD:R_0805_2012Metric -> Resistor_SMD:R_0603_1608Metric
- moved C19 200.6 mm to (114.5, 66.8), turned to 180 degrees
- moved C27 199.5 mm to (111.0, 78.2), turned to 180 degrees
- moved C21 194.2 mm to (120.9, 72.0), turned to 180 degrees
- moved U6 189.0 mm to (120.7, 67.0), turned to 90 degrees
- moved C15 185.5 mm to (130.5, 73.8), turned to -90 degrees
- moved C18 185.3 mm to (115.1, 64.9), turned to 180 degrees
- moved C17 184.8 mm to (114.5, 67.8), turned to 180 degrees
- moved C16 184.2 mm to (126.5, 66.5)
- moved U7 184.2 mm to (117.1, 75.9), turned to 180 degrees
- moved C22 182.7 mm to (118.7, 72.0)
- moved H2 181.6 mm to (101.6, 113.2)
- moved H3 181.2 mm to (101.3, 76.7)
- moved C26 180.8 mm to (115.1, 62.9), turned to 180 degrees
- moved J4 178.7 mm to (149.1, 51.8)
- moved C14 175.8 mm to (124.6, 73.8), turned to -90 degrees
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Connections:
- J2 pad 1: /rp2040/GPIO12 -> unconnected-(J2-Pad1)
- J2 pad 2: /rp2040/GPIO13 -> unconnected-(J2-Pad2)
- J2 pad 3: /rp2040/GPIO14 -> unconnected-(J2-Pad3)
- J2 pad 4: /rp2040/GPIO15 -> unconnected-(J2-Pad4)
- J2 pad 5: /rp2040/GPIO16 -> unconnected-(J2-Pad5)
- J2 pad 6: /rp2040/GPIO17 -> unconnected-(J2-Pad6)
- U6 pad 11: INT -> /rp2040/GPIO8
- U6 pad 12: AMP_BCLK -> /rp2040/GPIO9
- U6 pad 13: AMP_LRCLK -> /rp2040/GPIO10
- U6 pad 14: AMP_DIN -> /rp2040/GPIO11
- U6 pad 2: SD_MISO -> /rp2040/GPIO0
- U6 pad 29: /rp2040/GPIO18 -> AMP_BCLK
- U6 pad 3: SD_CS -> /rp2040/GPIO1
- U6 pad 30: /rp2040/GPIO19 -> AMP_LRCLK
- U6 pad 31: /rp2040/GPIO20 -> AMP_DIN
- U6 pad 32: /rp2040/GPIO21 -> RP2040_SDA
- U6 pad 34: /rp2040/GPIO22 -> RP2040_SCL
- U6 pad 35: /rp2040/GPIO23 -> INT
- U6 pad 36: /rp2040/GPIO24 -> SD_MISO
- U6 pad 37: /rp2040/GPIO25 -> SD_CS
- U6 pad 38: /rp2040/GPIO26_ADC0 -> SD_CLK
- U6 pad 39: /rp2040/GPIO27_ADC1 -> SD_MOSI
- U6 pad 4: SD_CLK -> /rp2040/GPIO2
- U6 pad 40: /rp2040/GPIO28_ADC2 -> SD_DAT1
- U6 pad 41: /rp2040/GPIO29_ADC3 -> SD_DAT2
- U6 pad 5: SD_MOSI -> /rp2040/GPIO3
- U6 pad 6: SD_DAT1 -> /rp2040/GPIO4
- U6 pad 7: SD_DAT2 -> /rp2040/GPIO5
- U6 pad 8: RP2040_SDA -> /rp2040/GPIO6
- U6 pad 9: RP2040_SCL -> /rp2040/GPIO7
Routing:
- net (no net): track 0.00 -> 26.8 mm
- net /USB_D-: track 0.00 -> 12.5 mm
- net /USB_D+: track 0.00 -> 10.5 mm
Other:
- board outline added: 100.5 x 70.6 mm
