File: src/kicad/board/board.kicad_pcb (KiCad board)
At the start: 2 copper layers, 100.5 x 70.6 mm, 82 parts, among them J1 USB_C_Receptacle_USB2.0, J2 Conn_01x06, J3 Micro_SD_Card_Det, J4 Conn_01x05_Male, J5 Conn_01x05_Male, J6 PWR_EN, J7 Screw_Terminal_Speaker, Q1 DMG2305UX, SW1 SW_Keyboard, SW2 SW_Keyboard, SW3 RotEncoder_S, SW4 SW_Keyboard, SW5 SW_Keyboard, SW6 BOOTSEL, U1 MCP23017_ML, U2 BQ25172, U3 TLV61070A, U4 XC6206P332MR, U5 MAX98357, U6 RP2040, U7 W25Q128JVS, Y1 X322512MSB4SI

Commit message: update
Parts:
- moved D4 66.0 mm to (128.7, 77.3), turned to 180 degrees
- moved Q1 65.2 mm to (134.8, 77.1), turned to 90 degrees
- moved L1 62.1 mm to (143.9, 71.4), turned to -90 degrees
- moved J6 61.0 mm to (170.7, 75.0)
- moved U3 60.2 mm to (150.4, 71.5), turned to 90 degrees
- moved C5 57.9 mm to (147.6, 71.2), turned to -90 degrees
- moved C6 56.8 mm to (153.1, 71.5), turned to -90 degrees
- moved D5 55.1 mm to (146.8, 66.6)
- moved R15 54.5 mm to (153.9, 68.2), turned to 90 degrees
- moved U2 54.4 mm to (139.2, 66.0)
- moved R16 53.8 mm to (143.1, 64.6), turned to 90 degrees
- moved C9 52.4 mm to (154.0, 65.4)
- moved R12 50.7 mm to (134.0, 66.1), turned to 90 degrees
- moved R13 50.2 mm to (146.6, 64.6)
- moved C8 49.9 mm to (153.7, 59.7)
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Routing:
- net Net-(BT1-Pad1): track 0.00 -> 52.3 mm, vias 0 -> 1
- net RP2040_SCL: track 0.00 -> 40.9 mm, vias 0 -> 2
- net GND: track 0.00 -> 39.0 mm, vias 0 -> 21
- net INT: track 0.00 -> 38.0 mm
- net RP2040_SDA: track 0.00 -> 37.8 mm
- net /USB_VBUS: track 0.00 -> 37.1 mm
- net Net-(J6-Pad2): track 0.00 -> 35.2 mm
- net /rp2040/QSPI_SS: track 0.00 -> 27.9 mm, vias 0 -> 2
- net (no net): track 26.8 -> 0.00 mm
- net /rp2040/~{USB_BOOT}: track 0.00 -> 18.9 mm, vias 0 -> 2
- net +3.3V: track 0.00 -> 18.5 mm
- net /USB_D-: track 12.5 -> 0.00 mm
- net /rp2040/QSPI_SD3: track 0.00 -> 11.9 mm, vias 0 -> 2
- net /rp2040/QSPI_SD1: track 0.00 -> 11.3 mm
- net Net-(C14-Pad2): track 0.00 -> 10.8 mm
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- added copper zone on F.Cu, net +3.3V
- added copper zone on B.Cu, net GND
