File: src/kicad/board/board.kicad_pcb (KiCad board)
At the start: 2 copper layers, 100 x 34 mm, 68 parts, among them J1 USB_C_Receptacle_USB2.0, J3 Micro_SD_Card_Det, J4 Conn_01x05_Male, J6 Conn_02x02_Top_Bottom, J7 Screw_Terminal_Speaker, Q1 DMG2305UX, SW6 BOOTSEL, U2 BQ25172, U3 TLV61070A, U4 XC6206P332MR, U5 MAX98357, U6 RP2040, U7 W25Q128JVS, Y1 X322512MSB4SI

Commit message: finish
Parts:
- moved L1 1.72 mm to (145.0, 82.8)
- moved C5 1.60 mm to (148.6, 82.5)
- moved U3 1.39 mm to (151.2, 82.8)
- moved C6 1.34 mm to (153.9, 82.8)
- moved R11 0.98 mm to (136.1, 77.3)
- moved R12 0.84 mm to (134.4, 77.3)
- moved R17 0.63 mm to (143.0, 78.4)
- moved R15 0.13 mm to (153.4, 79.5)
Routing:
- net GND: track 85.0 -> 90.3 mm, vias 50 -> 52
- net /Power/BAT_OR_USB_POWER_IN: track 53.1 -> 49.9 mm
- net VDD: track 41.8 -> 38.7 mm
- net Net-(R11-Pad2): track 2.87 -> 1.85 mm
- net Net-(BT1-Pad1): track 69.1 -> 68.2 mm
- net Net-(R16-Pad1): track 5.82 -> 6.63 mm
- net Net-(L1-Pad2): track 6.52 -> 5.74 mm
- net Net-(R12-Pad2): track 4.63 -> 3.91 mm
