File: src/kicad/board/power.kicad_sch (KiCad schematic)
At the start: 14 parts

Commit message: update pcb
Parts:
- added D1: D_Schottky, symbol Device:D_Schottky
- added Q1: DMG2301L, Package_TO_SOT_SMD:SOT-23, symbol Transistor_FET:DMG2301L
- U3: renamed from U?; footprint (none) -> Library:XB8089D
- gave numbers to parts that had none: 13
Connections:
- net BAT+: now also D1.2 (A), Q1.3 (D)
- net 5V_IN renamed PI_VBUS
- net PI_VBUS: now also Q1.1 (G)
- new net PI_VSYS: D1.1 (K), Q1.2 (S)
Other:
- moved on the sheet: BT1, C7, C8, C9, D2, D3, R10, R11, R12, R13, R8, R9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

Commit message: cleanup
Parts:
- removed BT1: Battery_Cell, symbol Device:Battery_Cell
- removed D1: D_Schottky, symbol Device:D_Schottky
- removed D2: PG, symbol Device:LED
- removed D3: CHRG, symbol Device:LED
- removed R10, R8: 1K, symbol Device:R
- removed R9: 536R, symbol Device:R
- removed U3: XB8089D, Library:XB8089D, symbol project_library:XB8089D
- removed U4: BQ24090DGQ, Package_SO:HVSSOP-10-1EP_3x3mm_P0.5mm_EP1.57x1.88mm_ThermalVias, symbol Battery_Management:BQ24090DGQ
- added BT1: 3 cell NiMH, Battery:BatteryHolder_Keystone_2462_2xAA, symbol Device:Battery
- added C4, C5: 10uF, Capacitor_SMD:C_0603_1608Metric, symbol Device:C
- added C6: 22uF, Capacitor_SMD:C_0603_1608Metric, symbol Device:C
- added D4: B5819W SL, Diode_SMD:D_SOD-123, symbol Diode:1N5819
- added D5: CHARGE_LED, LED_SMD:LED_0805_2012Metric, symbol Device:LED
- added J6: PWR_EN, Connector_PinHeader_2.54mm:PinHeader_1x02_P2.54mm_Vertical, symbol Connector_Generic:Conn_01x02
- added L1: 2.2uH, Inductor_SMD:L_Sunlord_MWSA05xxS, symbol Device:L
- added R14: 24.3K, Resistor_SMD:R_0805_2012Metric, symbol Device:R
- added R15: 2K7, Resistor_SMD:R_0603_1608Metric, symbol Device:R
- added R16, R17: 27K, Resistor_SMD:R_0603_1608Metric, symbol Device:R
- added U2: BQ25172, Package_SON:WSON-8-1EP_2x2mm_P0.5mm_EP0.9x1.6mm, symbol project_library:BQ25172
- added U3: TLV61070A, Package_SO:TSOP-6_1.65x3.05mm_P0.95mm, symbol project_library:TLV61070A
- added U4: XC6206P332MR, Package_TO_SOT_SMD:SOT-23-3, symbol Regulator_Linear:XC6206PxxxMR
- C7, C8, C9: value 0.1uF -> 10uF; footprint (none) -> Capacitor_SMD:C_0603_1608Metric; Vendor (none) -> C19702
- Q1: value DMG2301L -> DMG2305UX; Vendor (none) -> C2940629
- R11: value 10K -> 1K; footprint (none) -> Resistor_SMD:R_0603_1608Metric; Vendor (none) -> C21190
- R12: value 1K5 -> 10K; footprint (none) -> Resistor_SMD:R_0603_1608Metric; Vendor (none) -> C25804
- R13: value 1K5 -> 2K7; footprint (none) -> Resistor_SMD:R_0603_1608Metric; Vendor (none) -> C13167
Connections:
- net GND: now also C7.2, R12.1, BT1.2 (-), C4.2, C5.2, C6.2, R15.2, R16.2, R17.2, U2.4 (GND), U2.9 (PAD), U3.2 (GND), U4.1 (GND)
- net at R13.2: now also D5.2 (A)
- net at C7.1: now also Q1.3 (D), BT1.1 (+), U2.8 (OUT)
- net at R11.2: now also U2.2 (ISET)
- net at R12.2: now also U2.3 (TS)
- removed net BAT+: C9.1, Q1.3 (D), R12.1, R13.1
- net PI_VBUS: no longer names the net of Q1.1 (G)
- net PI_VBUS: now also R13.1, C4.1, D4.1 (K), U2.1 (IN); no longer C8.1
- net PI_VSYS: no longer names the net of Q1.2 (S)
- net PI_VSYS: now also J6.2 (Pin_2)
- new net: R17.1, U2.7 (VSET)
- new net: R14.2, R15.1, U3.4 (FB)
- new net: D5.1 (K), U2.5 (STAT)
- new net: L1.2, U3.1 (SW)
- new net: R16.1, U2.6 (TMR)
- new net 3.3V_OUT: C9.1, U4.2 (VO)
- new net 5V_OUT: C6.1, C8.1, R14.1, U3.5 (VOUT), U4.3 (VI)
- new net BAT_OR_USB_POWER: C5.1, J6.1 (Pin_1), L1.1, U3.3 (EN), U3.6 (VIN)
- new net USB_VBUS: D4.2 (A)
Other:
- note added: "27K -> 2-cell + intermittent charge"
- note added: "TODO: reduce coil whine"
- note added: "https://datasheets.raspberrypi.com/pico/pico-datasheet.pdf#powerchain-section"
- note removed: "TODO: confirm ISET, ISET2, and PRETERM R values"
- note removed: "https://s3.eu-central-1.amazonaws.com/elektormagazine/shopify/v59F5q8B9WcWKokvP9xom4TwesJ5q1NQ.pdf"
- note removed: "https://www.eevblog.com/forum/projects/problem-with-bq29700-battery-protection-ic/"
- note removed: "https://www.ti.com/lit/ds/symlink/bq24092.pdf?ts=1708754201508"

Commit message: update
Parts:
- removed J6: PWR_EN, Connector_PinHeader_2.54mm:PinHeader_1x02_P2.54mm_Vertical, symbol Connector_Generic:Conn_01x02
Connections:
- net BAT_OR_USB_POWER_OUT: now reaches Q1.2 (S)
- net BAT_OR_USB_POWER renamed BAT_OR_USB_POWER_IN
Changed lines of the file:
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@@
-    (stroke (width 0) (type default) (color 0 0 0 0))
-  )
-  (wire (pts (xy 201.93 72.39) (xy 213.36 72.39))
     (stroke (width 0) (type default) (color 0 0 0 0))
   )
@@
     (effects (font (size 1.27 1.27) italic) (justify left bottom))
   )
-  (label "BAT_OR_USB_POWER" (at 107.95 100.33 180)
-    (effects (font (size 1.27 1.27)) (justify right bottom))
-  )
-  (label "BAT_OR_USB_POWER" (at 213.36 72.39 0)
-    (effects (font (size 1.27 1.27)) (justify left bottom))
-  )
   (hierarchical_label "3.3V_OUT" (shape output) (at 204.47 132.08 0)
     (effects (font (size 1.27 1.27)) (justify left))
@@
   )
   (hierarchical_label "USB_VBUS" (shape input) (at 88.9 45.72 180)
+    (effects (font (size 1.27 1.27)) (justify right))
+  )
+  (hierarchical_label "BAT_OR_USB_POWER_OUT" (shape output) (at 199.39 72.39 0)
+    (effects (font (size 1.27 1.27)) (justify left))
+  )
+  (hierarchical_label "BAT_OR_USB_POWER_IN" (shape input) (at 107.95 100.33 180)
     (effects (font (size 1.27 1.27)) (justify right))
   )
@@
       (effects (font (size 1.27 1.27)) hide)
     )
-    (pin "1")
-    (pin "2")
-  )
-  (symbol (lib_id "Connector_Generic:Conn_01x02") (at 201.93 77.47 270) (unit 1)
-    (in_bom yes) (on_board yes) (fields_autoplaced)
-    (property "Reference" "J6" (id 0) (at 204.47 76.1999 90)
-      (effects (font (size 1.27 1.27)) (justify left))
-    )
-    (property "Value" "PWR_EN" (id 1) (at 204.47 78.7399 90)
-      (effects (font (size 1.27 1.27)) (justify left))
-    )
-    (property "Footprint" "Connector_PinHeader_2.54mm:PinHeader_1x02_P2.54mm_Vertical" (id 2) (at 201.93 77.47 0)
-      (effects (font (size 1.27 1.27)) hide)
-    )
-    (property "Datasheet" "~" (id 3) (at 201.93 77.47 0)
-      (effects (font (size 1.27 1.27)) hide)
-    )

Commit message: updated with new pcb
Other:
- note added: "6 hours"
- note added: "TODO: iset may be too high"
Changed lines of the file:
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@@
     (stroke (width 0) (type default) (color 0 0 0 0))
+  )
+  (text "TODO: iset may be too high\n" (at 111.76 71.12 0)
+    (effects (font (size 1.27 1.27)) (justify left bottom))
   )
   (text "TODO: reduce coil whine" (at 125.73 134.62 0)
     (effects (font (size 1.27 1.27)) (justify left bottom))
   )
-  (text "27K -> 2-cell + intermittent charge\n" (at 158.75 73.66 90)
-    (effects (font (size 1.27 1.27)) (justify left bottom))
+  (text "27K -> 2-cell + intermittent charge\n" (at 184.15 77.47 180)
+    (effects (font (size 1.27 1.27)) (justify right bottom))
   )
   (text "https://datasheets.raspberrypi.com/pico/pico-datasheet.pdf#powerchain-section"
@@
     (effects (font (size 1.27 1.27) italic) (justify left bottom))
   )
+  (text "6 hours\n" (at 146.05 62.23 0)
+    (effects (font (size 1.27 1.27)) (justify left bottom))
+  )
   (hierarchical_label "3.3V_OUT" (shape output) (at 204.47 132.08 0)
