File: src/kicad/board/board.kicad_sch (KiCad schematic)
At the start: 19 parts, among them J1 USB_C_Receptacle_USB2.0, J3 Micro_SD_Card_Det, J4 Conn_01x05_Male

Commit message: update
Parts:
- added J6: Conn_02x02_Top_Bottom, Connector_PinHeader_2.54mm:PinHeader_2x02_P2.54mm_Vertical, symbol Connector_Generic:Conn_02x02_Top_Bottom
Connections:
- net rp2040/SWCLK: now also J6.1 (Pin_1)
- net rp2040/SWD: now also J6.2 (Pin_2)
- new net Power/BAT_OR_USB_POWER_IN: J6.4 (Pin_4)
- new net Power/BAT_OR_USB_POWER_OUT: J6.3 (Pin_3)
- no-connect marks 24 -> 22
Other:
- sheet Power ports: added BAT_OR_USB_POWER_IN, BAT_OR_USB_POWER_OUT; removed none
- note removed: "TODO: optimize pin config"
Changed lines of the file:
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@@
   (no_connect (at 81.28 173.99))
   (no_connect (at 111.76 101.6))
-  (no_connect (at 129.54 48.26))
   (no_connect (at 148.59 83.82))
   (no_connect (at 148.59 81.28))
@@
   (no_connect (at 148.59 60.96))
   (no_connect (at 148.59 76.2))
-  (no_connect (at 127 48.26))
   (no_connect (at 148.59 68.58))
   (no_connect (at 52.07 72.39))
@@
     (stroke (width 0) (type default) (color 0 0 0 0))
   )
-  (wire (pts (xy 194.31 57.15) (xy 212.09 57.15))
-    (stroke (width 0) (type default) (color 0 0 0 0))
-  )
   (wire (pts (xy 74.93 142.24) (xy 74.93 137.16))
     (stroke (width 0) (type default) (color 0 0 0 0))
   )
+  (wire (pts (xy 162.56 36.83) (xy 162.56 62.23))
+    (stroke (width 0) (type default) (color 0 0 0 0))
+  )
   (wire (pts (xy 72.39 36.83) (xy 72.39 39.37))
     (stroke (width 0) (type default) (color 0 0 0 0))
@@
     (stroke (width 0) (type default) (color 0 0 0 0))
   )
+  (wire (pts (xy 161.29 39.37) (xy 161.29 64.77))
+    (stroke (width 0) (type default) (color 0 0 0 0))
+  )
+  (wire (pts (xy 179.07 64.77) (xy 204.47 64.77))
+    (stroke (width 0) (type default) (color 0 0 0 0))
+  )
   (wire (pts (xy 52.07 41.91) (xy 54.61 41.91))
     (stroke (width 0) (type default) (color 0 0 0 0))
@@
     (stroke (width 0) (type default) (color 0 0 0 0))
   )
-  (wire (pts (xy 209.55 50.8) (xy 212.09 50.8))
+  (wire (pts (xy 209.55 41.91) (xy 212.09 41.91))
     (stroke (width 0) (type default) (color 0 0 0 0))
   )
@@
     (stroke (width 0) (type default) (color 0 0 0 0))
   )
+  (wire (pts (xy 203.2 46.99) (xy 203.2 62.23))
+    (stroke (width 0) (type default) (color 0 0 0 0))
+  )
   (wire (pts (xy 77.47 149.86) (xy 77.47 156.21))
     (stroke (width 0) (type default) (color 0 0 0 0))
@@
     (stroke (width 0) (type default) (color 0 0 0 0))
   )
+  (wire (pts (xy 127 48.26) (xy 127 36.83))
+    (stroke (width 0) (type default) (color 0 0 0 0))
+  )
   (wire (pts (xy 72.39 137.16) (xy 74.93 137.16))
     (stroke (width 0) (type default) (color 0 0 0 0))
@@
     (stroke (width 0) (type default) (color 0 0 0 0))
   )
+  (wire (pts (xy 203.2 62.23) (xy 179.07 62.23))
+    (stroke (width 0) (type default) (color 0 0 0 0))
+  )
   (wire (pts (xy 52.07 54.61) (xy 52.07 57.15))
     (stroke (width 0) (type default) (color 0 0 0 0))
   )
+  (wire (pts (xy 161.29 64.77) (xy 166.37 64.77))
+    (stroke (width 0) (type default) (color 0 0 0 0))
+  )
   (wire (pts (xy 73.66 163.83) (xy 73.66 173.99))
     (stroke (width 0) (type default) (color 0 0 0 0))
   )
-  (wire (pts (xy 194.31 55.88) (xy 194.31 57.15))
-    (stroke (width 0) (type default) (color 0 0 0 0))
-  )
   (wire (pts (xy 106.68 76.2) (xy 111.76 76.2))
     (stroke (width 0) (type default) (color 0 0 0 0))
@@
     (stroke (width 0) (type default) (color 0 0 0 0))
   )
+  (wire (pts (xy 241.3 59.69) (xy 250.19 59.69))
+    (stroke (width 0) (type default) (color 0 0 0 0))
+  )
   (wire (pts (xy 74.93 57.15) (xy 74.93 72.39))
     (stroke (width 0) (type default) (color 0 0 0 0))
@@
     (stroke (width 0) (type default) (color 0 0 0 0))
   )
+  (wire (pts (xy 212.09 46.99) (xy 203.2 46.99))
+    (stroke (width 0) (type default) (color 0 0 0 0))
+  )
   (wire (pts (xy 54.61 41.91) (xy 54.61 36.83))
     (stroke (width 0) (type default) (color 0 0 0 0))
@@
     (stroke (width 0) (type default) (color 0 0 0 0))
   )
+  (wire (pts (xy 250.19 59.69) (xy 250.19 55.88))
+    (stroke (width 0) (type default) (color 0 0 0 0))
+  )
   (wire (pts (xy 106.68 83.82) (xy 111.76 83.82))
     (stroke (width 0) (type default) (color 0 0 0 0))
@@
     (stroke (width 0) (type default) (color 0 0 0 0))
   )
+  (wire (pts (xy 204.47 50.8) (xy 212.09 50.8))
+    (stroke (width 0) (type default) (color 0 0 0 0))
+  )
+  (wire (pts (xy 127 36.83) (xy 162.56 36.83))
+    (stroke (width 0) (type default) (color 0 0 0 0))
+  )
   (wire (pts (xy 81.28 166.37) (xy 44.45 166.37))
     (stroke (width 0) (type default) (color 0 0 0 0))
@@
     (stroke (width 0) (type default) (color 0 0 0 0))
   )
+  (wire (pts (xy 129.54 48.26) (xy 129.54 39.37))
+    (stroke (width 0) (type default) (color 0 0 0 0))
+  )
   (wire (pts (xy 39.37 167.64) (xy 44.45 167.64))
     (stroke (width 0) (type default) (color 0 0 0 0))
@@
     (stroke (width 0) (type default) (color 0 0 0 0))
   )
+  (wire (pts (xy 204.47 64.77) (xy 204.47 50.8))
+    (stroke (width 0) (type default) (color 0 0 0 0))
+  )
   (wire (pts (xy 36.83 80.01) (xy 36.83 82.55))
     (stroke (width 0) (type default) (color 0 0 0 0))
@@
   )
   (wire (pts (xy 67.31 142.24) (xy 67.31 137.16))
+    (stroke (width 0) (type default) (color 0 0 0 0))
+  )
+  (wire (pts (xy 162.56 62.23) (xy 166.37 62.23))
+    (stroke (width 0) (type default) (color 0 0 0 0))
+  )
+  (wire (pts (xy 129.54 39.37) (xy 161.29 39.37))
     (stroke (width 0) (type default) (color 0 0 0 0))
   )
@@
     (effects (font (size 1.27 1.27)) (justify left bottom))
   )
-  (text "TODO: optimize pin config\n" (at 123.19 46.99 0)
-    (effects (font (size 1.27 1.27) italic) (justify left bottom))
-  )
   (text "connect to ground with resistor\n\nhttps://www.reddit.com/r/PrintedCircuitBoard/comments/18tr602/review_request_rp2040_breakout_board/#lightbox\nhttps://www.synopsys.com/designware-ip/technical-bulletin/converting-existing-designs.html"
     (at -20.32 -22.86 0)
@@
     (effects (font (size 1.27 1.27)) (justify left bottom))
   )
-  (label "USB_VBUS" (at 209.55 50.8 180)
+  (label "USB_VBUS" (at 209.55 41.91 180)
     (effects (font (size 1.27 1.27)) (justify right bottom))
   )
@@
     (pin "5")
   )
-  (symbol (lib_id "power:+3.3V") (at 194.31 55.88 0) (unit 1)
+  (symbol (lib_id "power:+3.3V") (at 250.19 55.88 0) (unit 1)
     (in_bom yes) (on_board yes) (fields_autoplaced)
-    (property "Reference" "#PWR08" (id 0) (at 194.31 59.69 0)
-      (effects (font (size 1.27 1.27)) hide)
-    )
-    (property "Value" "+3.3V" (id 1) (at 194.31 50.8 0))
-    (property "Footprint" "" (id 2) (at 194.31 55.88 0)
-      (effects (font (size 1.27 1.27)) hide)
-    )
-    (property "Datasheet" "" (id 3) (at 194.31 55.88 0)
+    (property "Reference" "#PWR08" (id 0) (at 250.19 59.69 0)
+      (effects (font (size 1.27 1.27)) hide)
+    )
+    (property "Value" "+3.3V" (id 1) (at 250.19 50.8 0))
+    (property "Footprint" "" (id 2) (at 250.19 55.88 0)
+      (effects (font (size 1.27 1.27)) hide)
+    )
+    (property "Datasheet" "" (id 3) (at 250.19 55.88 0)
       (effects (font (size 1.27 1.27)) hide)
     )
@@
       (effects (font (size 1.27 1.27)) hide)
     )
+  )
+  (symbol (lib_id "Connector_Generic:Conn_02x02_Top_Bottom") (at 171.45 62.23 0) (unit 1)
+    (in_bom yes) (on_board yes) (fields_autoplaced)
+    (property "Reference" "J6" (id 0) (at 172.72 55.88 0))
+    (property "Value" "Conn_02x02_Top_Bottom" (id 1) (at 172.72 58.42 0))
+    (property "Footprint" "Connector_PinHeader_2.54mm:PinHeader_2x02_P2.54mm_Vertical" (id 2) (at 171.45 62.23 0)
+      (effects (font (size 1.27 1.27)) hide)
+    )
+    (property "Datasheet" "~" (id 3) (at 171.45 62.23 0)
+      (effects (font (size 1.27 1.27)) hide)
+    )
+    (pin "1")
+    (pin "2")
+    (pin "3")
+    (pin "4")
   )
   (symbol (lib_id "Device:R") (at 60.96 68.58 0) (unit 1)
@@
     (pin "2")
   )
-  (sheet (at 212.09 46.99) (size 19.05 15.24) (fields_autoplaced)
+  (sheet (at 212.09 39.37) (size 29.21 22.86) (fields_autoplaced)
     (stroke (width 0.1524) (type solid) (color 0 0 0 0))
     (fill (color 0 0 0 0.0000))
-    (property "Sheet name" "Power" (id 0) (at 212.09 46.2784 0)
+    (property "Sheet name" "Power" (id 0) (at 212.09 38.6584 0)
       (effects (font (size 1.27 1.27)) (justify left bottom))
     )
@@
       (effects (font (size 1.27 1.27)) (justify left top))
     )
-    (pin "3.3V_OUT" output (at 212.09 57.15 180)
-      (effects (font (size 1.27 1.27)) (justify left))
+    (pin "3.3V_OUT" output (at 241.3 59.69 0)
+      (effects (font (size 1.27 1.27)) (justify right))
     )
     (pin "5V_OUT" output (at 212.09 59.69 180)
       (effects (font (size 1.27 1.27)) (justify left))
     )
-    (pin "USB_VBUS" input (at 212.09 50.8 180)
+    (pin "USB_VBUS" input (at 212.09 41.91 180)
+      (effects (font (size 1.27 1.27)) (justify left))
+    )
+    (pin "BAT_OR_USB_POWER_OUT" output (at 212.09 46.99 180)
+      (effects (font (size 1.27 1.27)) (justify left))
+    )
+    (pin "BAT_OR_USB_POWER_IN" input (at 212.09 50.8 180)
       (effects (font (size 1.27 1.27)) (justify left))
     )
@@
       (reference "J4") (unit 1) (value "Conn_01x05_Male") (footprint "Connector_JST:JST_PH_B5B-PH-SM4-TB_1x05-1MP_P2.00mm_Vertical")
     )
-    (path "/4532e7a8-aa46-45fe-9bdb-5c2c6a438547/517bbb0c-4128-41ca-81cf-f67870dfe288"
-      (reference "J6") (unit 1) (value "PWR_EN") (footprint "Connector_PinHeader_2.54mm:PinHeader_1x02_P2.54mm_Vertical")
+    (path "/bacaf2d5-6169-4e5e-83cb-be4c6836c7f5"
+      (reference "J6") (unit 1) (value "Conn_02x02_Top_Bottom") (footprint "Connector_PinHeader_2.54mm:PinHeader_2x02_P2.54mm_Vertical")
     )
     (path "/d540bb9b-d45f-4ddd-b651-2c00d8abffca/d8757b13-5fcb-40e0-8b42-9b760e31dbf2"

Commit message: finish
Other:
- note added: "make sure these pins correspond with these pins: https://datasheets.raspberrypi.com/rp2040/rp2040-datasheet.pdf#%5B%7B%22num%22%3A16%2C%22gen%22%3A0%7D%2C%7B%22name%22%3A%22XYZ%22%7D%2C115%2C625.392%2Cnull%5D"
Changed lines of the file:
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@@
     (effects (font (size 1.27 1.27) italic) (justify left bottom))
+  )
+  (text "make sure these pins correspond with these pins:\nhttps://datasheets.raspberrypi.com/rp2040/rp2040-datasheet.pdf#%5B%7B%22num%22%3A16%2C%22gen%22%3A0%7D%2C%7B%22name%22%3A%22XYZ%22%7D%2C115%2C625.392%2Cnull%5D"
+    (at -6.35 213.36 0)
+    (effects (font (size 1.27 1.27)) (justify left bottom))
   )
   (text "https://cdn-learn.adafruit.com/downloads/pdf/adafruit-microsd-spi-sdio.pdf"
