File: src/kicad/io-board/io-board.kicad_pcb (KiCad board)
At the start: 2 copper layers, 100 x 34 mm, 10 parts, among them J1 Conn_01x05_Male, SW1 SW_Keyboard, SW2 SW_Keyboard, SW3 RotEncoder_S, SW4 SW_Keyboard, SW5 SW_Keyboard, U1 MCP23017_ML

Commit message: update
Other:
- board text added: "IO Board V0.2"
