File: src/kicad/io-board/io-board.kicad_sch (KiCad schematic)
At the start: 10 parts, among them J1 Conn_01x05_Male, SW1 SW_Keyboard, SW2 SW_Keyboard, SW3 RotEncoder_S, SW4 SW_Keyboard, SW5 SW_Keyboard, U1 MCP23017_ML

Commit message: update
Parts:
- SW1, SW2, SW4, SW5: Vendor (none) -> C5156480
Changed lines of the file:
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@@
+      (effects (font (size 1.27 1.27)) hide)
+    )
+    (property "Vendor" "C5156480" (id 4) (at 151.13 69.85 0)
       (effects (font (size 1.27 1.27)) hide)
     )
@@
     )
     (property "Datasheet" "~" (id 3) (at 177.8 64.77 0)
+      (effects (font (size 1.27 1.27)) hide)
+    )
+    (property "Vendor" "C5156480" (id 4) (at 177.8 69.85 0)
       (effects (font (size 1.27 1.27)) hide)
     )
@@
       (effects (font (size 1.27 1.27)) hide)
     )
+    (property "Vendor" "C5156480" (id 4) (at 151.13 54.61 0)
+      (effects (font (size 1.27 1.27)) hide)
+    )
     (pin "1")
     (pin "2")
@@
       (effects (font (size 1.27 1.27)) hide)
     )
+    (property "Vendor" "C5156480" (id 4) (at 177.8 54.61 0)
+      (effects (font (size 1.27 1.27)) hide)
+    )
