File: pcb/io-board/io-board.kicad_pcb (KiCad board)
At the start: 2 copper layers, 100 x 34 mm, 10 parts, among them J1 Conn_01x05_Male, SW1 SW_Keyboard, SW2 SW_Keyboard, SW3 RotEncoder_S, SW4 SW_Keyboard, SW5 SW_Keyboard, U1 MCP23017_ML

Commit message: pcb version 0.3
Parts:
- added D1: LED, LED_SMD:LED_0805_2012Metric, F.Cu at (109.9, 102.1)
- added D2: LED, LED_SMD:LED_0805_2012Metric, F.Cu at (114.9, 102.1)
- added D3: LED, LED_SMD:LED_0805_2012Metric, F.Cu at (119.9, 102.1)
- added D4: LED, LED_SMD:LED_0805_2012Metric, F.Cu at (124.9, 102.1)
- added D5: LED, LED_SMD:LED_0805_2012Metric, F.Cu at (129.9, 102.1)
- added D6: LED, LED_SMD:LED_0805_2012Metric, F.Cu at (134.9, 102.1)
- added D7: LED, LED_SMD:LED_0805_2012Metric, F.Cu at (139.9, 102.1)
- added D8: LED, LED_SMD:LED_0805_2012Metric, F.Cu at (144.9, 102.1)
- added JP1: Jumper_2_Bridged, Jumper:SolderJumper-2_P1.3mm_Bridged_RoundedPad1.0x1.5mm, F.Cu at (116.2, 93.2)
- added JP2: Jumper_2_Bridged, Jumper:SolderJumper-2_P1.3mm_Bridged_RoundedPad1.0x1.5mm, F.Cu at (118.8, 93.2)
- added JP3: Jumper_2_Bridged, Jumper:SolderJumper-2_P1.3mm_Bridged_RoundedPad1.0x1.5mm, F.Cu at (121.4, 93.2)
- added JP4: Jumper_2_Bridged, Jumper:SolderJumper-2_P1.3mm_Bridged_RoundedPad1.0x1.5mm, F.Cu at (124.0, 93.2)
- added JP5: Jumper_2_Bridged, Jumper:SolderJumper-2_P1.3mm_Bridged_RoundedPad1.0x1.5mm, F.Cu at (126.6, 93.2)
- added JP6: Jumper_2_Bridged, Jumper:SolderJumper-2_P1.3mm_Bridged_RoundedPad1.0x1.5mm, F.Cu at (129.2, 93.2)
- added JP7: Jumper_2_Bridged, Jumper:SolderJumper-2_P1.3mm_Bridged_RoundedPad1.0x1.5mm, F.Cu at (131.8, 93.2)
- added JP8: Jumper_2_Bridged, Jumper:SolderJumper-2_P1.3mm_Bridged_RoundedPad1.0x1.5mm, F.Cu at (134.4, 93.2)
- added R1: 2K7, Resistor_SMD:R_0603_1608Metric, F.Cu at (116.5, 97.7)
- added R2: 2K7, Resistor_SMD:R_0603_1608Metric, F.Cu at (118.7, 97.7)
- added R3: 2K7, Resistor_SMD:R_0603_1608Metric, F.Cu at (120.8, 97.7)
- added R4: 2K7, Resistor_SMD:R_0603_1608Metric, F.Cu at (122.9, 97.7)
- added R5: 2K7, Resistor_SMD:R_0603_1608Metric, F.Cu at (125.0, 97.7)
- added R6: 2K7, Resistor_SMD:R_0603_1608Metric, F.Cu at (127.1, 97.7)
- added R7: 2K7, Resistor_SMD:R_0603_1608Metric, F.Cu at (129.3, 97.7)
- added R8: 2K7, Resistor_SMD:R_0603_1608Metric, F.Cu at (131.5, 97.7)
- moved SW3 0.83 mm to (186.8, 93.5)
Connections:
- U1 pad 17: unconnected-(U1-Pad17) -> Net-(JP8-Pad2)
- U1 pad 18: unconnected-(U1-Pad18) -> Net-(JP7-Pad2)
- U1 pad 19: unconnected-(U1-Pad19) -> Net-(JP6-Pad2)
- U1 pad 20: unconnected-(U1-Pad20) -> Net-(JP5-Pad2)
- U1 pad 21: unconnected-(U1-Pad21) -> Net-(JP4-Pad2)
- U1 pad 22: unconnected-(U1-Pad22) -> Net-(JP3-Pad2)
- U1 pad 23: unconnected-(U1-Pad23) -> Net-(JP2-Pad2)
- U1 pad 24: unconnected-(U1-Pad24) -> Net-(JP1-Pad2)
Routing:
- net Net-(JP6-Pad2): track 0.00 -> 60.9 mm, vias 0 -> 2
- net Net-(JP1-Pad2): track 0.00 -> 57.9 mm, vias 0 -> 2
- net Net-(JP2-Pad2): track 0.00 -> 56.3 mm, vias 0 -> 2
- net Net-(JP7-Pad2): track 0.00 -> 56.1 mm, vias 0 -> 2
- net Net-(JP3-Pad2): track 0.00 -> 54.8 mm, vias 0 -> 2
- net Net-(JP4-Pad2): track 0.00 -> 53.7 mm, vias 0 -> 2
- net Net-(JP5-Pad2): track 0.00 -> 51.9 mm, vias 0 -> 2
- net Net-(JP8-Pad2): track 0.00 -> 51.5 mm, vias 0 -> 2
- net Net-(D8-Pad2): track 0.00 -> 15.8 mm
- net Net-(D7-Pad2): track 0.00 -> 13.0 mm
- net GND: track 32.6 -> 44.9 mm, vias 9 -> 17
- net Net-(D6-Pad2): track 0.00 -> 10.2 mm
- net Net-(D5-Pad2): track 0.00 -> 7.33 mm
- net Net-(D1-Pad2): track 0.00 -> 7.14 mm
- net Net-(D4-Pad2): track 0.00 -> 4.85 mm
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
Commit message: pcb v0.3
Other:
- board text added: "IO Board V0.3"
- board text removed: "IO Board V0.2"
Changed lines of the file:
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@@
   (gr_arc (start 197.872598 100.71) (mid 197.140365 102.477767) (end 195.372598 103.21) (layer "Edge.Cuts") (width 0.1))
   (gr_arc (start 97.872598 71.21) (mid 98.458384 69.795786) (end 99.872598 69.21) (layer "Edge.Cuts") (width 0.1))
-  (gr_text "IO Board V0.2" (at 181.3 98.6) (layer "F.SilkS")
+  (gr_text "IO Board V0.3" (at 183.65 99.7) (layer "F.SilkS")
     (effects (font (size 1 1) (thickness 0.15)))
   )

Commit message: update io pcb
Parts:
- SW1, SW2, SW4, SW5: footprint Library:Kailh_socket_MX -> Button_Switch_Keyboard:SW_Cherry_MX_1.00u_PCB
- moved SW2 4.91 mm to (151.9, 81.3)
- moved SW4 4.91 mm to (132.7, 81.3)
- moved SW1 4.91 mm to (171.1, 81.3)
- moved SW5 4.91 mm to (113.5, 81.3)
Routing:
- net B3: track 69.3 -> 57.7 mm
- net B2: track 50.1 -> 39.2 mm
- net GND: track 44.9 -> 37.0 mm, vias 17 -> 13
- net B1: track 31.1 -> 24.1 mm
Other:
- board text added: "IO Board V0.4"
- board text removed: "IO Board V0.3"
