File: pcb/io-board/io-board.kicad_sch (KiCad schematic)
At the start: 10 parts, among them J1 Conn_01x05_Male, SW1 SW_Keyboard, SW2 SW_Keyboard, SW3 RotEncoder_S, SW4 SW_Keyboard, SW5 SW_Keyboard, U1 MCP23017_ML

Commit message: pcb version 0.3
Parts:
- added D1, D2, D3, D4, D5, D6, D7, D8: LED, LED_SMD:LED_0805_2012Metric, symbol Device:LED
- added JP1, JP2, JP3, JP4, JP5, JP6, JP7, JP8: Jumper_2_Bridged, Jumper:SolderJumper-2_P1.3mm_Bridged_RoundedPad1.0x1.5mm, symbol Jumper:Jumper_2_Bridged
- added R1, R2, R3, R4, R5, R6, R7, R8: 2K7, Resistor_SMD:R_0603_1608Metric, symbol Device:R
Connections:
- net GND: now also D1.1 (K), D2.1 (K), D3.1 (K), D4.1 (K), D5.1 (K), D6.1 (K), D7.1 (K), D8.1 (K)
- net at U1.17 (GPA0): now also JP8.2 (B)
- net at U1.18 (GPA1): now also JP7.2 (B)
- net at U1.19 (GPA2): now also JP6.2 (B)
- net at U1.20 (GPA3): now also JP5.2 (B)
- net at U1.21 (GPA4): now also JP4.2 (B)
- net at U1.22 (GPA5): now also JP3.2 (B)
- net at U1.23 (GPA6): now also JP2.2 (B)
- net at U1.24 (GPA7): now also JP1.2 (B)
- new net: JP7.1 (A), R7.1
- new net: D7.2 (A), R7.2
- new net: JP6.1 (A), R6.1
- new net: D5.2 (A), R5.2
- new net: D8.2 (A), R8.2
- new net: JP8.1 (A), R8.1
- new net: D1.2 (A), R1.2
- new net: D6.2 (A), R6.2
- new net: JP3.1 (A), R3.1
- new net: JP2.1 (A), R2.1
- new net: D2.2 (A), R2.2
- new net: JP1.1 (A), R1.1
- new net: D4.2 (A), R4.2
- new net: JP5.1 (A), R5.1
- new net: JP4.1 (A), R4.1
- new net: D3.2 (A), R3.2
- no-connect marks 10 -> 2
Other:
- moved on the sheet: J1, SW1, SW2, SW3, SW4, SW5

Commit message: update io pcb
Parts:
- SW1, SW2, SW4, SW5: footprint Library:Kailh_socket_MX -> Button_Switch_Keyboard:SW_Cherry_MX_1.00u_PCB; Vendor C5156480 -> (none)
Changed lines of the file:
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@@
     (property "Reference" "SW2" (id 0) (at 140.97 41.91 0))
     (property "Value" "SW_Keyboard" (id 1) (at 140.97 44.45 0))
-    (property "Footprint" "Library:Kailh_socket_MX" (id 2) (at 142.24 44.45 0)
+    (property "Footprint" "Button_Switch_Keyboard:SW_Cherry_MX_1.00u_PCB" (id 2) (at 142.24 44.45 0)
       (effects (font (size 1.27 1.27)) hide)
     )
@@
       (effects (font (size 1.27 1.27)) hide)
     )
-    (property "Vendor" "C5156480" (id 4) (at 142.24 49.53 0)
+    (property "Vendor" "" (id 4) (at 142.24 49.53 0)
       (effects (font (size 1.27 1.27)) hide)
     )
@@
     (property "Reference" "SW5" (id 0) (at 165.1 41.91 0))
     (property "Value" "SW_Keyboard" (id 1) (at 165.1 44.45 0))
-    (property "Footprint" "Library:Kailh_socket_MX" (id 2) (at 168.91 44.45 0)
+    (property "Footprint" "Button_Switch_Keyboard:SW_Cherry_MX_1.00u_PCB" (id 2) (at 168.91 44.45 0)
       (effects (font (size 1.27 1.27)) hide)
     )
@@
       (effects (font (size 1.27 1.27)) hide)
     )
-    (property "Vendor" "C5156480" (id 4) (at 168.91 49.53 0)
+    (property "Vendor" "" (id 4) (at 168.91 49.53 0)
       (effects (font (size 1.27 1.27)) hide)
     )
@@
     (property "Reference" "SW1" (id 0) (at 139.7 26.67 0))
     (property "Value" "SW_Keyboard" (id 1) (at 139.7 29.21 0))
-    (property "Footprint" "Library:Kailh_socket_MX" (id 2) (at 142.24 29.21 0)
+    (property "Footprint" "Button_Switch_Keyboard:SW_Cherry_MX_1.00u_PCB" (id 2) (at 142.24 29.21 0)
       (effects (font (size 1.27 1.27)) hide)
     )
@@
       (effects (font (size 1.27 1.27)) hide)
     )
-    (property "Vendor" "C5156480" (id 4) (at 142.24 34.29 0)
+    (property "Vendor" "" (id 4) (at 142.24 34.29 0)
       (effects (font (size 1.27 1.27)) hide)
     )
@@
     (property "Reference" "SW4" (id 0) (at 165.1 26.67 0))
     (property "Value" "SW_Keyboard" (id 1) (at 165.1 29.21 0))
-    (property "Footprint" "Library:Kailh_socket_MX" (id 2) (at 168.91 29.21 0)
+    (property "Footprint" "Button_Switch_Keyboard:SW_Cherry_MX_1.00u_PCB" (id 2) (at 168.91 29.21 0)
       (effects (font (size 1.27 1.27)) hide)
     )
@@
       (effects (font (size 1.27 1.27)) hide)
     )
-    (property "Vendor" "C5156480" (id 4) (at 168.91 34.29 0)
+    (property "Vendor" "" (id 4) (at 168.91 34.29 0)
       (effects (font (size 1.27 1.27)) hide)
     )
@@
     )
     (path "/38d62497-788e-4ff6-8fcf-2d3156dab531"
-      (reference "SW1") (unit 1) (value "SW_Keyboard") (footprint "Library:Kailh_socket_MX")
+      (reference "SW1") (unit 1) (value "SW_Keyboard") (footprint "Button_Switch_Keyboard:SW_Cherry_MX_1.00u_PCB")
     )
     (path "/0904299e-addd-41f7-b087-37c7d5d4d25c"
-      (reference "SW2") (unit 1) (value "SW_Keyboard") (footprint "Library:Kailh_socket_MX")
+      (reference "SW2") (unit 1) (value "SW_Keyboard") (footprint "Button_Switch_Keyboard:SW_Cherry_MX_1.00u_PCB")
     )
     (path "/b0319775-902d-430c-adb5-99ce41a419be"
@@
     )
     (path "/53e68fbf-6c77-43ee-a781-dcdeeb9859d1"
-      (reference "SW4") (unit 1) (value "SW_Keyboard") (footprint "Library:Kailh_socket_MX")
+      (reference "SW4") (unit 1) (value "SW_Keyboard") (footprint "Button_Switch_Keyboard:SW_Cherry_MX_1.00u_PCB")
     )
     (path "/0a6f416c-01fa-4a9c-bf19-9ccb29c102f6"
-      (reference "SW5") (unit 1) (value "SW_Keyboard") (footprint "Library:Kailh_socket_MX")
+      (reference "SW5") (unit 1) (value "SW_Keyboard") (footprint "Button_Switch_Keyboard:SW_Cherry_MX_1.00u_PCB")
     )
     (path "/166cff32-c1ba-4296-9dde-75e01fb4e6b3"
